Commit message: Arm working on Gazebo!

File: thorp_bringup/urdf/thorp_gazebo.urdf.xacro (robot description, xacro)
@@ -138,4 +138,9 @@
   <Sharp_GP2Y0A21_IR_sim name="r155"/>
   <!-- Gazebo configuration for other structural parts -->
+  <gazebo reference="sonars_mount_link">
+    <material>Gazebo/Black</material>
+    <selfCollide>true</selfCollide>
+    <gravity>true</gravity>
+  </gazebo>
   <gazebo reference="senz3d_mount_link">
     <material>Gazebo/Black</material>
@@ -143,8 +148,29 @@
     <gravity>true</gravity>
   </gazebo>
-  <gazebo reference="opencm_joint_link">
+  <gazebo reference="opencm_link">
     <material>Gazebo/Black</material>
     <selfCollide>true</selfCollide>
     <gravity>true</gravity>
   </gazebo>
+  <!-- Gazebo configuration for arm control -->
+  <gazebo>
+    <plugin name="gazebo_ros_control" filename="libgazebo_ros_control.so"/>
+  </gazebo>
+  <AX12_transmission name="arm_shoulder_pan"/>
+  <AX12_transmission name="arm_shoulder_lift"/>
+  <AX12_transmission name="arm_elbow_flex"/>
+  <AX12_transmission name="arm_wrist_flex"/>
+  <AX12_transmission name="gripper"/>
+  <xacro:macro name="AX12_transmission" params="name">
+    <transmission name="${name}_trans">
+      <type>transmission_interface/SimpleTransmission</type>
+      <joint name="${name}_joint">
+        <hardwareInterface>EffortJointInterface</hardwareInterface>
+      </joint>
+      <actuator name="${name}_motor">
+        <hardwareInterface>EffortJointInterface</hardwareInterface>
+        <mechanicalReduction>1</mechanicalReduction>
+      </actuator>
+    </transmission>
+  </xacro:macro>
 </robot>
