Commit message: Update to reflect the new configurable turtlebot arm stuff

File: thorp_bringup/urdf/standalone_arm.urdf.xacro (robot description, xacro)
@@ -5,5 +5,5 @@
     xmlns:interface="http://playerstage.sourceforge.net/gazebo/xmlschema/#interface">
     <!-- Included URDF Files -->
-    <xacro:include filename="$(find turtlebot_arm_description)/urdf/arm.xacro" />
+    <xacro:include filename="$(find turtlebot_arm_description)/urdf/turtlebot_arm.xacro" />
     <!-- As we don't have here a turtlebot, add a base_link link as its location reference -->
     <link name="base_link"/>
@@ -11,6 +11,15 @@
          for the first joint (arm_shoulder_pan) to allow accessing to different operational
          areas, e.g. left handed vs. right handed robot -->
-    <turtlebot_arm parent="base_link" color="white" gripper_color="green"
-                   joints_vlimit="0.3571" pan_llimit="-4.189" pan_ulimit="1.047">
+    <xacro:property name="joints_vlimit" value="0.3571"/>
+    <xacro:property name="pan_llimit" value="-4.189"/>
+    <xacro:property name="pan_ulimit" value="1.047"/>
+    <xacro:property name="shoulder_llimit" value="-2.617"/>
+    <xacro:property name="shoulder_ulimit" value="2.617"/>
+    <xacro:property name="elbow_llimit" value="-2.617"/>
+    <xacro:property name="elbow_ulimit" value="2.617"/>
+    <xacro:property name="wrist_llimit" value="-1.745"/>
+    <xacro:property name="wrist_ulimit" value="1.745"/>
+    <turtlebot_arm parent="base_link" color="white" gripper_color="Green"
+                   pincher_gripper="false" turtlebot_gripper="true">
       <!-- Place the "floating" arm at the location it should be if mounted on a turtlebot,
            as pick and place and other demos assume this location -->

File: thorp_bringup/urdf/thorp.urdf.xacro (robot description, xacro)
@@ -13,5 +13,5 @@
 <robot name="Thorp" xmlns:xacro="http://ros.org/wiki/xacro">
   <xacro:include filename="$(find turtlebot_description)/urdf/turtlebot_library.urdf.xacro"/>
-  <xacro:include filename="$(find turtlebot_arm_description)/urdf/arm.xacro"/>
+  <xacro:include filename="$(find turtlebot_arm_description)/urdf/turtlebot_arm.xacro"/>
   <xacro:include filename="$(find thorp_bringup)/urdf/thorp_gazebo.urdf.xacro"/>
   <xacro:include filename="$(find softkinetic_camera)/urdf/senz3d.urdf.xacro"/>
@@ -22,7 +22,17 @@
   <!-- Turtlebot arm, its controller board and its mounting on Thorp -->
   <!-- Note that the arm position is biased to the left of the robot, and the dead angle also
-       points to the left; with this configuration, the arm can reach most of the top plate -->
+       points to the left; with this configuration, the arm can reach most of the top plate.
+       We also use a deliberately low joints velocity limit to improve safety and precision -->
+  <xacro:property name="joints_vlimit" value="0.3571"/>
+  <xacro:property name="pan_llimit" value="-4.189"/>
+  <xacro:property name="pan_ulimit" value="1.047"/>
+  <xacro:property name="shoulder_llimit" value="-2.617"/>
+  <xacro:property name="shoulder_ulimit" value="2.617"/>
+  <xacro:property name="elbow_llimit" value="-2.617"/>
+  <xacro:property name="elbow_ulimit" value="2.617"/>
+  <xacro:property name="wrist_llimit" value="-1.745"/>
+  <xacro:property name="wrist_ulimit" value="1.745"/>
   <turtlebot_arm parent="plate_top_link" color="White" gripper_color="Black"
-                 joints_vlimit="0.3571" pan_llimit="-4.189" pan_ulimit="1.047">
+                 pincher_gripper="false" turtlebot_gripper="true">
     <origin xyz="0.10914 0.0295 0.0284"/>
   </turtlebot_arm>

Commit message: Remove the robot arm's right-handed configuration, making the arm shoulder pan servo point to the front instead to the right.

File: thorp_bringup/urdf/standalone_arm.urdf.xacro (robot description, xacro)
@@ -12,12 +12,12 @@
          areas, e.g. left handed vs. right handed robot -->
     <xacro:property name="joints_vlimit" value="0.3571"/>
-    <xacro:property name="pan_llimit" value="-4.189"/>
-    <xacro:property name="pan_ulimit" value="1.047"/>
+    <xacro:property name="pan_llimit" value="-2.617"/>
+    <xacro:property name="pan_ulimit" value=" 2.617"/>
     <xacro:property name="shoulder_llimit" value="-2.617"/>
-    <xacro:property name="shoulder_ulimit" value="2.617"/>
+    <xacro:property name="shoulder_ulimit" value=" 2.617"/>
     <xacro:property name="elbow_llimit" value="-2.617"/>
-    <xacro:property name="elbow_ulimit" value="2.617"/>
+    <xacro:property name="elbow_ulimit" value=" 2.617"/>
     <xacro:property name="wrist_llimit" value="-1.745"/>
-    <xacro:property name="wrist_ulimit" value="1.745"/>
+    <xacro:property name="wrist_ulimit" value=" 1.745"/>
     <turtlebot_arm parent="base_link" color="white" gripper_color="Green"
                    pincher_gripper="false" turtlebot_gripper="true">

File: thorp_bringup/urdf/thorp.urdf.xacro (robot description, xacro)
@@ -21,16 +21,17 @@
   <sensor_kinect  parent="base_link"/>
   <!-- Turtlebot arm, its controller board and its mounting on Thorp -->
-  <!-- Note that the arm position is biased to the left of the robot, and the dead angle also
-       points to the left; with this configuration, the arm can reach most of the top plate.
+  <!-- Note that the arm position is biased to the left of the robot, while the Senz3D camera
+       is biased to the right; with this configuration, the arm lefts doesn't block completely
+       camera view to the operation space.
        We also use a deliberately low joints velocity limit to improve safety and precision -->
   <xacro:property name="joints_vlimit" value="0.3571"/>
-  <xacro:property name="pan_llimit" value="-4.189"/>
-  <xacro:property name="pan_ulimit" value="1.047"/>
+  <xacro:property name="pan_llimit" value="-2.617"/>
+  <xacro:property name="pan_ulimit" value=" 2.617"/>
   <xacro:property name="shoulder_llimit" value="-2.617"/>
-  <xacro:property name="shoulder_ulimit" value="2.617"/>
+  <xacro:property name="shoulder_ulimit" value=" 2.617"/>
   <xacro:property name="elbow_llimit" value="-2.617"/>
-  <xacro:property name="elbow_ulimit" value="2.617"/>
+  <xacro:property name="elbow_ulimit" value=" 2.617"/>
   <xacro:property name="wrist_llimit" value="-1.745"/>
-  <xacro:property name="wrist_ulimit" value="1.745"/>
+  <xacro:property name="wrist_ulimit" value=" 1.745"/>
   <turtlebot_arm parent="plate_top_link" color="White" gripper_color="Black"
                  pincher_gripper="false" turtlebot_gripper="true">
