Commit message: Properly configure Kinect + Asus Xtion Pro for simulation

File: thorp_bringup/urdf/kinect.urdf.xacro (robot description, xacro)
@@ -1,5 +1,4 @@
 <?xml version="1.0"?>
 <robot name="kinect_camera" xmlns:xacro="http://ros.org/wiki/xacro">
-  <xacro:include filename="$(find turtlebot_description)/urdf/turtlebot_gazebo.urdf.xacro"/>
   <xacro:include filename="$(find turtlebot_description)/urdf/turtlebot_properties.urdf.xacro"/>
   <xacro:property name="kinect_cam_py" value="-0.0125"/>
@@ -60,6 +59,6 @@
 	</joint>
 	<link name="${name}_depth_optical_frame"/>
-	<!-- Kinect sensor for simulation -->
-	<turtlebot_sim_3dsensor/>
+    <!-- RGBD sensor for simulation -->
+    <thorp_sim_3dsensor name="${name}" depth_registration="false"/>
   </xacro:macro>
 </robot>

File: thorp_bringup/urdf/thorp_gazebo.urdf.xacro (robot description, xacro)
@@ -1,6 +1,53 @@
 <?xml version="1.0"?>
 <robot name="thorp_gazebo" xmlns:xacro="http://ros.org/wiki/xacro">
+  <!-- Simulated Microsoft Kinect / ASUS Xtion PRO Live macros; included on their respective xacro files -->
+  <xacro:macro name="thorp_sim_3dsensor" params="name depth_registration">
+    <gazebo reference="${name}_link">
+      <sensor type="depth" name="${name}">
+        <always_on>true</always_on>
+        <update_rate>20.0</update_rate>
+        <camera>
+          <horizontal_fov>${60.0*M_PI/180.0}</horizontal_fov>
+          <image>
+            <format>B8G8R8</format>
+            <width>640</width>
+            <height>480</height>
+          </image>
+          <clip>
+            <near>0.05</near>
+            <far>8.0</far>
+          </clip>
+        </camera>
+        <plugin name="kinect_camera_controller" filename="libgazebo_ros_openni_kinect.so">
+          <cameraName>${name}</cameraName>
+          <alwaysOn>true</alwaysOn>
+          <updateRate>10</updateRate>
+          <imageTopicName>rgb/image_raw</imageTopicName>
+          <cameraInfoTopicName>rgb/camera_info</cameraInfoTopicName>
+          <xacro:if value="${depth_registration}">  <!-- Normally for manipulation camera (Xtion) -->
+            <depthImageTopicName>depth_registered/image_raw</depthImageTopicName>
+            <pointCloudTopicName>depth_registered/points</pointCloudTopicName>
+            <depthImageCameraInfoTopicName>depth_registered/camera_info</depthImageCameraInfoTopicName>
+          </xacro:if>
+          <xacro:unless value="${depth_registration}">  <!-- Normally for navigation camera (Kinect) -->
+            <depthImageTopicName>depth/image_raw</depthImageTopicName>
+            <pointCloudTopicName>depth/points</pointCloudTopicName>
+            <depthImageCameraInfoTopicName>depth/camera_info</depthImageCameraInfoTopicName>
+          </xacro:unless>
+          <frameName>${name}_rgb_optical_frame</frameName>  <!-- TODO confirm -->
+          <baseline>0.1</baseline>
+          <distortion_k1>0.0</distortion_k1>
+          <distortion_k2>0.0</distortion_k2>
+          <distortion_k3>0.0</distortion_k3>
+          <distortion_t1>0.0</distortion_t1>
+          <distortion_t2>0.0</distortion_t2>
+          <pointCloudCutoff>0.4</pointCloudCutoff>
+          <pointCloudCutoffMax>6.0</pointCloudCutoffMax>
+        </plugin>
+      </sensor>
+    </gazebo>
+  </xacro:macro>
   <!-- Simulated Creative Senz3d camera -->
-  <gazebo reference="senz3d_camera_link">
+  <gazebo reference="senz3d_link">
     <sensor type="depth" name="senz3d">
       <always_on>true</always_on>
@@ -27,5 +74,5 @@
         <cameraInfoTopicName>rgb/camera_info</cameraInfoTopicName>
         <depthImageCameraInfoTopicName>depth/camera_info</depthImageCameraInfoTopicName>
-        <frameName>senz3d_camera_gazebo_optical_frame</frameName>
+        <frameName>senz3d_gazebo_optical_frame</frameName>
         <baseline>0.1</baseline>
         <distortion_k1>0.0</distortion_k1>
@@ -34,5 +81,6 @@
         <distortion_t1>0.0</distortion_t1>
         <distortion_t2>0.0</distortion_t2>
-        <pointCloudCutoff>0.15</pointCloudCutoff>
+        <pointCloudCutoff>0.10</pointCloudCutoff>
+        <pointCloudCutoffMax>1.0</pointCloudCutoffMax>
       </plugin>
     </sensor>
@@ -154,4 +202,9 @@
     <gravity>true</gravity>
   </gazebo>
+  <gazebo reference="xtion_mount_link">
+    <material>Gazebo/Black</material>
+    <selfCollide>true</selfCollide>
+    <gravity>true</gravity>
+  </gazebo>
   <gazebo reference="opencm_link">
     <material>Gazebo/Black</material>

File: thorp_bringup/urdf/xtion.urdf.xacro (robot description, xacro)
@@ -1,6 +1,4 @@
 <?xml version="1.0"?>
 <robot name="xtion_camera" xmlns:xacro="http://ros.org/wiki/xacro">
-  <xacro:include filename="$(find turtlebot_description)/urdf/turtlebot_gazebo.urdf.xacro"/>
-  <!-- <xacro:include filename="$(find turtlebot_description)/urdf/turtlebot_properties.urdf.xacro"/> -->
   <!-- Xacro properties -->
   <xacro:property name="asus_xtion_pro_depth_rel_rgb_py" value="0.0270"/>
@@ -28,5 +26,6 @@
     <link name="${name}_link">
       <visual>
-        <origin xyz="0.0 0.0035 0.0375" rpy="0 0 0"/>
+        <origin xyz="-0.015 0.0035 0.004" rpy="0 0 0"/>
+        <!-- <origin xyz="0.0 0.0035 0.0375" rpy="0 0 0"/>    a OJO -->
         <geometry>
           <mesh filename="package://turtlebot_description/meshes/sensors/xtion_pro_camera.dae"/>
@@ -59,33 +58,6 @@
     </joint>
     <link name="${name}_depth_optical_frame"/>
-    <!-- RGBD sensor for simulation, same as Kinect
-    <turtlebot_sim_3dsensor/> TODO  no vale... usa la pose dada x el fichero de calib -->
-    <!-- Asus mount
-    <joint name="mount_asus_xtion_pro_joint" type="fixed">
-      <origin xyz="-0.1024 0.0 0.272" rpy="0 0 0"/>
-      <parent link="${parent}"/>
-      <child link="mount_asus_xtion_pro_link"/>
-    </joint>
-    <link name="mount_asus_xtion_pro_link">
-      <visual>
-        <origin xyz="0 0 0" rpy="${-M_PI/2} 0 0"/>
-        <geometry>
-          <mesh filename="package://turtlebot_description/meshes/sensors/xtion_pro_stack.dae"/>
-        </geometry>
-      </visual>
-      <collision>
-        <origin xyz="0.0 0.0 0.0" rpy="0 0 0" />
-        <geometry>
-        <box size="0.0330 0.2760 0.0120"/>
-      </geometry>
-      </collision>
-      <inertial>
-        <mass value="0.170" />
-        <origin xyz="0 0 0" />
-        <inertia ixx="0.001152600" ixy="0.0" ixz="0.0"
-                 iyy="0.000148934" iyz="0.0"
-                 izz="0.001154654" />
-      </inertial>
-    </link>-->
+    <!-- RGBD sensor for simulation -->
+    <thorp_sim_3dsensor name="${name}" depth_registration="true"/>
   </xacro:macro>
 </robot>
