Commit message: Add TB arm

File: thorp_bringup/urdf/thorp.urdf.xacro (robot description, xacro)
@@ -11,7 +11,20 @@
 <robot name="turtlebot" xmlns:xacro="http://ros.org/wiki/xacro">
   <xacro:include filename="$(find turtlebot_description)/urdf/turtlebot_library.urdf.xacro"/>
+  <xacro:include filename="$(find turtlebot_arm_description)/urdf/arm.xacro"/>
+  <!-- Plain Turtlebot -->
   <kobuki/>
   <stack_hexagons parent="base_link"/>
   <sensor_kinect  parent="base_link"/>
+  <!-- Turtlebot arm plus mounting on Thorp -->
+  <turtlebot_arm parent="base_link" color="white" gripper_color="black">
+    <origin xyz="0.0985 0.0295 0.425"/>
+  </turtlebot_arm>
+  <arm_mount parent="arm_base_link" name="arm_mount" color="black">
+    <origin xyz="0 0 0" rpy="0 0 0" />
+  </arm_mount>
+  <stack_bottom_pole parent="arm_base_link" number="10" x_loc= "0.0" y_loc= "0.0288" z_loc="-0.0112"/>
+  <stack_bottom_pole parent="arm_base_link" number="11" x_loc= "0.0" y_loc= "-0.0288" z_loc="-0.0112"/>
+  <stack_bottom_pole parent="arm_base_link" number="12" x_loc= "-0.038" y_loc= "-0.0288" z_loc="-0.0112"/>
+  <stack_bottom_pole parent="arm_base_link" number="13" x_loc= "-0.038" y_loc= "0.0288" z_loc="-0.0112"/>
   <!-- Sonar links forming a half ring centered on (and slightly above) base_link-->
   <joint name="s_m90_joint" type="fixed">

Commit message: Merely cosmetic

File: thorp_bringup/urdf/thorp.urdf.xacro (robot description, xacro)
@@ -8,9 +8,10 @@
     - 11 sonar links
     - 4 IR sensor links
+    - Turtlebot arm
 -->
 <robot name="turtlebot" xmlns:xacro="http://ros.org/wiki/xacro">
   <xacro:include filename="$(find turtlebot_description)/urdf/turtlebot_library.urdf.xacro"/>
   <xacro:include filename="$(find turtlebot_arm_description)/urdf/arm.xacro"/>
-  <!-- Plain Turtlebot -->
+  <!-- Plain Turtlebot 2 -->
   <kobuki/>
   <stack_hexagons parent="base_link"/>
@@ -21,10 +22,10 @@
   </turtlebot_arm>
   <arm_mount parent="arm_base_link" name="arm_mount" color="black">
-    <origin xyz="0 0 0" rpy="0 0 0" />
+    <origin xyz="0.0 0.0 0.0" rpy="0.0 0.0 0.0"/>
   </arm_mount>
-  <stack_bottom_pole parent="arm_base_link" number="10" x_loc= "0.0" y_loc= "0.0288" z_loc="-0.0112"/>
-  <stack_bottom_pole parent="arm_base_link" number="11" x_loc= "0.0" y_loc= "-0.0288" z_loc="-0.0112"/>
+  <stack_bottom_pole parent="arm_base_link" number="10" x_loc= " 0.0"   y_loc= " 0.0288" z_loc="-0.0112"/>
+  <stack_bottom_pole parent="arm_base_link" number="11" x_loc= " 0.0"   y_loc= "-0.0288" z_loc="-0.0112"/>
   <stack_bottom_pole parent="arm_base_link" number="12" x_loc= "-0.038" y_loc= "-0.0288" z_loc="-0.0112"/>
-  <stack_bottom_pole parent="arm_base_link" number="13" x_loc= "-0.038" y_loc= "0.0288" z_loc="-0.0112"/>
+  <stack_bottom_pole parent="arm_base_link" number="13" x_loc= "-0.038" y_loc= " 0.0288" z_loc="-0.0112"/>
   <!-- Sonar links forming a half ring centered on (and slightly above) base_link-->
   <joint name="s_m90_joint" type="fixed">

Commit message: Place arm relative to top plate. Add tf for Senz3D camera

File: thorp_bringup/urdf/thorp.urdf.xacro (robot description, xacro)
@@ -9,6 +9,8 @@
     - 4 IR sensor links
     - Turtlebot arm
+    - Senz3D camera
 -->
 <robot name="turtlebot" xmlns:xacro="http://ros.org/wiki/xacro">
+  <xacro:property name="pi" value="3.1415926535897931"/>
   <xacro:include filename="$(find turtlebot_description)/urdf/turtlebot_library.urdf.xacro"/>
   <xacro:include filename="$(find turtlebot_arm_description)/urdf/arm.xacro"/>
@@ -18,6 +20,6 @@
   <sensor_kinect  parent="base_link"/>
   <!-- Turtlebot arm plus mounting on Thorp -->
-  <turtlebot_arm parent="base_link" color="white" gripper_color="black">
-    <origin xyz="0.0985 0.0295 0.425"/>
+  <turtlebot_arm parent="plate_top_link" color="white" gripper_color="black">
+    <origin xyz="0.11214 0.0295 0.0284"/>
   </turtlebot_arm>
   <arm_mount parent="arm_base_link" name="arm_mount" color="black">
@@ -28,4 +30,24 @@
   <stack_bottom_pole parent="arm_base_link" number="12" x_loc= "-0.038" y_loc= "-0.0288" z_loc="-0.0112"/>
   <stack_bottom_pole parent="arm_base_link" number="13" x_loc= "-0.038" y_loc= " 0.0288" z_loc="-0.0112"/>
+  <!-- Senz3D camera plus mounting on Thorp -->
+  <joint name="senz3d_camera_joint" type="fixed">
+    <origin xyz="-0.085 -0.082 0.28" rpy="${pi/2 + 0.907571211037} 0.0 ${pi/2}"/> <!-- 0,10471975512 -->
+    <parent link="plate_top_link"/>
+    <child link="senz3d_camera_link"/>
+  </joint>
+  <link name="senz3d_camera_link">
+<!--     <visual>
+      <origin xyz="0.0 0.0 0.0" rpy="0.0 0.0 0.0" />
+      <geometry>
+        <mesh filename="package://thorp_bringup/resources/meshes/senz3d.stl" scale="1.0 1.0 1.0"/>
+      </geometry>
+    </visual>
+    <collision>
+      <origin xyz="0.0 0.0 0.0" rpy="0.0 0.0 0.0" />
+      <geometry>
+        <box size="0.025 0.038 0.004"/>
+      </geometry>
+    </collision> TODO peta RViz-->
+  </link>
   <!-- Sonar links forming a half ring centered on (and slightly above) base_link-->
   <joint name="s_m90_joint" type="fixed">

Commit message: Add one middle pole to the Senz 3D height

File: thorp_bringup/urdf/thorp.urdf.xacro (robot description, xacro)
@@ -32,5 +32,5 @@
   <!-- Senz3D camera plus mounting on Thorp -->
   <joint name="senz3d_camera_joint" type="fixed">
-    <origin xyz="-0.085 -0.082 0.28" rpy="${pi/2 + 0.907571211037} 0.0 ${pi/2}"/> <!-- 0,10471975512 -->
+    <origin xyz="-0.085 -0.082 0.34" rpy="${pi/2 + 0.907571211037} 0.0 ${pi/2}"/> <!-- 0,10471975512 -->
     <parent link="plate_top_link"/>
     <child link="senz3d_camera_link"/>

Commit message: Add visual, collision, inertia and mounting for the Senz3D

File: thorp_bringup/urdf/thorp.urdf.xacro (robot description, xacro)
@@ -11,6 +11,5 @@
     - Senz3D camera
 -->
-<robot name="turtlebot" xmlns:xacro="http://ros.org/wiki/xacro">
-  <xacro:property name="pi" value="3.1415926535897931"/>
+<robot name="Thorp" xmlns:xacro="http://ros.org/wiki/xacro">
   <xacro:include filename="$(find turtlebot_description)/urdf/turtlebot_library.urdf.xacro"/>
   <xacro:include filename="$(find turtlebot_arm_description)/urdf/arm.xacro"/>
@@ -26,27 +25,72 @@
     <origin xyz="0.0 0.0 0.0" rpy="0.0 0.0 0.0"/>
   </arm_mount>
-  <stack_bottom_pole parent="arm_base_link" number="10" x_loc= " 0.0"   y_loc= " 0.0288" z_loc="-0.0112"/>
-  <stack_bottom_pole parent="arm_base_link" number="11" x_loc= " 0.0"   y_loc= "-0.0288" z_loc="-0.0112"/>
-  <stack_bottom_pole parent="arm_base_link" number="12" x_loc= "-0.038" y_loc= "-0.0288" z_loc="-0.0112"/>
-  <stack_bottom_pole parent="arm_base_link" number="13" x_loc= "-0.038" y_loc= " 0.0288" z_loc="-0.0112"/>
+  <stack_bottom_pole parent="arm_base_link" number="10" x_loc=" 0.0"   y_loc=" 0.0288" z_loc="-0.0112"/>
+  <stack_bottom_pole parent="arm_base_link" number="11" x_loc=" 0.0"   y_loc="-0.0288" z_loc="-0.0112"/>
+  <stack_bottom_pole parent="arm_base_link" number="12" x_loc="-0.038" y_loc="-0.0288" z_loc="-0.0112"/>
+  <stack_bottom_pole parent="arm_base_link" number="13" x_loc="-0.038" y_loc=" 0.0288" z_loc="-0.0112"/>
   <!-- Senz3D camera plus mounting on Thorp -->
+  <!-- Mounting poles: we emulate one top and two middle poles overlapping two top poles -->
+  <!-- The Z loc of the upper poles is : 1/2*plate height + 1/2*top pole height + 2*middle pole height (without screw) -->
+  <stack_top_pole parent="plate_top_link" number="10" x_loc="-0.1024" y_loc=" 0.098" z_loc="${0.006/2 + 0.2032/2}"/>
+  <stack_top_pole parent="plate_top_link" number="11" x_loc="-0.1024" y_loc="-0.098" z_loc="${0.006/2 + 0.2032/2}"/>
+  <stack_top_pole parent="plate_top_link" number="12" x_loc="-0.1024" y_loc=" 0.098" z_loc="${0.006/2 + 0.2032/2 + 0.1}"/>
+  <stack_top_pole parent="plate_top_link" number="13" x_loc="-0.1024" y_loc="-0.098" z_loc="${0.006/2 + 0.2032/2 + 0.1}"/>
+  <!-- Mounting plate; this structure is provisional -->
+  <joint name="senz3d_mount_joint" type="fixed">
+    <origin xyz="-0.1024 0.0 ${0.2032 + 0.006 + 0.1}" rpy="0.0 0.0 0.0"/>
+    <parent link="plate_top_link"/>
+    <child link="senz3d_mount_link"/>
+  </joint>
+  <link name="senz3d_mount_link">
+    <visual>
+      <origin xyz="0.0 0.0 0.0" rpy="0.0 0.0 0.0"/>
+      <geometry>
+        <box size="0.02 0.24 0.006"/>
+      </geometry>
+      <material name="black">
+        <color rgba="0.0 0.0 0.0 1.0"/>
+      </material>
+    </visual>
+    <collision>
+      <origin xyz="0.0 0.0 0.0" rpy="0.0 0.0 0.0"/>
+      <geometry>
+        <box size="0.02 0.24 0.006"/>
+      </geometry>
+    </collision>
+    <inertial>
+      <mass value="0.01"/>
+      <origin xyz="0 0 0"/>
+      <inertia ixx="0.001" ixy="0.0" ixz="0.0"
+        iyy="0.001" iyz="0.0"
+        izz="0.001"/>
+    </inertial>
+  </link>
+  <!-- Camera -->
   <joint name="senz3d_camera_joint" type="fixed">
-    <origin xyz="-0.085 -0.082 0.34" rpy="${pi/2 + 0.907571211037} 0.0 ${pi/2}"/> <!-- 0,10471975512 -->
+    <origin xyz="-0.065 -0.082 0.325" rpy="${M_PI/2 + 0.907571211037} 0.0 ${M_PI/2}"/>
     <parent link="plate_top_link"/>
     <child link="senz3d_camera_link"/>
   </joint>
   <link name="senz3d_camera_link">
-<!--     <visual>
-      <origin xyz="0.0 0.0 0.0" rpy="0.0 0.0 0.0" />
+    <visual>
+      <origin xyz="0.0 0.0 0.0" rpy="0.0 0.0 0.0"/>
       <geometry>
-        <mesh filename="package://thorp_bringup/resources/meshes/senz3d.stl" scale="1.0 1.0 1.0"/>
+        <!-- As we don't have a Senz3D mesh, use a deformed Asus Xtion Pro instead -->
+        <mesh filename="package://turtlebot_description/meshes/sensors/asus_xtion_pro_live.dae" scale="0.0006 0.0015 0.001"/>
       </geometry>
     </visual>
     <collision>
-      <origin xyz="0.0 0.0 0.0" rpy="0.0 0.0 0.0" />
+      <origin xyz="0.0 0.0 -0.005" rpy="0 0 0"/>
       <geometry>
-        <box size="0.025 0.038 0.004"/>
-      </geometry>
-    </collision> TODO peta RViz-->
+      <box size="0.11 0.04 0.04"/>
+    </geometry>
+    </collision>
+    <inertial>
+      <mass value="0.01"/>
+      <origin xyz="0 0 0"/>
+      <inertia ixx="0.001" ixy="0.0" ixz="0.0"
+        iyy="0.001" iyz="0.0"
+        izz="0.001"/>
+    </inertial>
   </link>
   <!-- Sonar links forming a half ring centered on (and slightly above) base_link-->

Commit message: Change the direction of the arm dead angle to the left.

File: thorp_bringup/urdf/thorp.urdf.xacro (robot description, xacro)
@@ -19,6 +19,8 @@
   <sensor_kinect  parent="base_link"/>
   <!-- Turtlebot arm plus mounting on Thorp -->
+  <!-- Note that the arm position is biased to the left of the robot, and the dead angle also
+       points to the left; with this configuration, the arm can reach most of the top plate -->
   <turtlebot_arm parent="plate_top_link" color="white" gripper_color="black"
-                 joints_vlimit="0.3571" pan_llimit="-1.047" pan_ulimit="4.189">
+                 joints_vlimit="0.3571" pan_llimit="-4.189" pan_ulimit="1.047">
     <origin xyz="0.11214 0.0295 0.0284"/>
   </turtlebot_arm>
@@ -69,5 +71,5 @@
   <!-- Camera -->
   <joint name="senz3d_camera_joint" type="fixed">
-    <origin xyz="-0.065 -0.082 0.325" rpy="${M_PI/2 + 0.907571211037} 0.0 ${M_PI/2}"/>
+    <origin xyz="-0.055 -0.062 0.355" rpy="${M_PI/2 + 0.907571211037} 0.0 ${M_PI/2}"/>
     <parent link="plate_top_link"/>
     <child link="senz3d_camera_link"/>

Commit message: Emulate the OpenCM9.04 as a box and other minor adjustements

File: thorp_bringup/urdf/thorp.urdf.xacro (robot description, xacro)
@@ -32,14 +32,44 @@
   <stack_bottom_pole parent="arm_base_link" number="12" x_loc="-0.038" y_loc="-0.0288" z_loc="-0.0112"/>
   <stack_bottom_pole parent="arm_base_link" number="13" x_loc="-0.038" y_loc=" 0.0288" z_loc="-0.0112"/>
+  <!-- Emulate the OpenCM9.04 as a box -->
+  <joint name="opencm_joint" type="fixed">
+    <origin xyz="0.045 0.03 0.008" rpy="0.0 0.0 0.0"/>
+    <parent link="plate_top_link"/>
+    <child link="opencm_joint_link"/>
+  </joint>
+  <link name="opencm_joint_link">
+    <visual>
+      <origin xyz="0.0 0.0 0.0" rpy="0.0 0.0 0.0"/>
+      <geometry>
+        <box size="0.027 0.0665 0.01"/>
+      </geometry>
+      <material name="green">
+        <color rgba="0.22 0.32 0.14 1.0"/>
+      </material>
+    </visual>
+    <collision>
+      <origin xyz="0.0 0.0 0.0" rpy="0.0 0.0 0.0"/>
+      <geometry>
+        <box size="0.027 0.0665 0.012"/>
+      </geometry>
+    </collision>
+    <inertial>
+      <mass value="0.01"/>
+      <origin xyz="0 0 0"/>
+      <inertia ixx="0.001" ixy="0.0" ixz="0.0"
+        iyy="0.001" iyz="0.0"
+        izz="0.001"/>
+    </inertial>
+  </link>
   <!-- Senz3D camera plus mounting on Thorp -->
   <!-- Mounting poles: we emulate one top and two middle poles overlapping two top poles -->
   <!-- The Z loc of the upper poles is : 1/2*plate height + 1/2*top pole height + 2*middle pole height (without screw) -->
-  <stack_top_pole parent="plate_top_link" number="10" x_loc="-0.1024" y_loc=" 0.098" z_loc="${0.006/2 + 0.2032/2}"/>
-  <stack_top_pole parent="plate_top_link" number="11" x_loc="-0.1024" y_loc="-0.098" z_loc="${0.006/2 + 0.2032/2}"/>
-  <stack_top_pole parent="plate_top_link" number="12" x_loc="-0.1024" y_loc=" 0.098" z_loc="${0.006/2 + 0.2032/2 + 0.1}"/>
-  <stack_top_pole parent="plate_top_link" number="13" x_loc="-0.1024" y_loc="-0.098" z_loc="${0.006/2 + 0.2032/2 + 0.1}"/>
+  <stack_top_pole parent="plate_top_link" number="10" x_loc="-0.0874" y_loc=" 0.098" z_loc="${0.006/2 + 0.2032/2}"/>
+  <stack_top_pole parent="plate_top_link" number="11" x_loc="-0.0874" y_loc="-0.098" z_loc="${0.006/2 + 0.2032/2}"/>
+  <stack_top_pole parent="plate_top_link" number="12" x_loc="-0.0874" y_loc=" 0.098" z_loc="${0.006/2 + 0.2032/2 + 0.1}"/>
+  <stack_top_pole parent="plate_top_link" number="13" x_loc="-0.0874" y_loc="-0.098" z_loc="${0.006/2 + 0.2032/2 + 0.1}"/>
   <!-- Mounting plate; this structure is provisional -->
   <joint name="senz3d_mount_joint" type="fixed">
-    <origin xyz="-0.1024 0.0 ${0.2032 + 0.006 + 0.1}" rpy="0.0 0.0 0.0"/>
+    <origin xyz="-0.0874 0.0 ${0.2032 + 0.006 + 0.1}" rpy="0.0 0.0 0.0"/>
     <parent link="plate_top_link"/>
     <child link="senz3d_mount_link"/>
@@ -71,5 +101,5 @@
   <!-- Camera -->
   <joint name="senz3d_camera_joint" type="fixed">
-    <origin xyz="-0.055 -0.062 0.355" rpy="${M_PI/2 + 0.907571211037} 0.0 ${M_PI/2}"/>
+    <origin xyz="-0.045 -0.062 0.345" rpy="${M_PI/2 + 0.907571211037} 0.0 ${M_PI/2}"/>
     <parent link="plate_top_link"/>
     <child link="senz3d_camera_link"/>

Commit message: Add frames for RGB and depth optical axes

File: thorp_bringup/urdf/thorp.urdf.xacro (robot description, xacro)
@@ -101,5 +101,6 @@
   <!-- Camera -->
   <joint name="senz3d_camera_joint" type="fixed">
-    <origin xyz="-0.045 -0.062 0.345" rpy="${M_PI/2 + 0.907571211037} 0.0 ${M_PI/2}"/>
+    <!-- <origin xyz="-0.045 -0.062 0.345" rpy="${M_PI/2 + 0.907571211037} 0.0 ${M_PI/2}"/> -->
+    <origin xyz="-0.0552702 -0.0411472 0.323393" rpy="2.3447 0.0160734 1.59265"/>
     <parent link="plate_top_link"/>
     <child link="senz3d_camera_link"/>
@@ -120,5 +121,5 @@
     </collision>
     <inertial>
-      <mass value="0.01"/>
+      <mass value="0.271"/>
       <origin xyz="0 0 0"/>
       <inertia ixx="0.001" ixy="0.0" ixz="0.0"
@@ -127,4 +128,29 @@
     </inertial>
   </link>
+  <!-- Add frames for RGB and depth optical axes -->
+  <joint name="senz3d_rgb_joint" type="fixed">
+    <origin xyz="0.0125 0.0 0.0" rpy="0.0 0.0 0.0"/>
+    <parent link="senz3d_camera_link"/>
+    <child link="senz3d_rgb_frame"/>
+  </joint>
+  <link name="senz3d_rgb_frame"/>
+  <joint name="senz3d_rgb_optical_joint" type="fixed">
+    <origin xyz="0.0 0.0 0.0" rpy="0.0 0.0 ${M_PI}" />
+    <parent link="senz3d_rgb_frame"/>
+    <child link="senz3d_rgb_optical_frame"/>
+  </joint>
+  <link name="senz3d_rgb_optical_frame"/>
+  <joint name="senz3d_depth_joint" type="fixed">
+    <origin xyz="-0.0125 0.0 0.0" rpy="0.0 0.0 0.0"/>
+    <parent link="senz3d_camera_link"/>
+    <child link="senz3d_depth_frame"/>
+  </joint>
+  <link name="senz3d_depth_frame"/>
+  <joint name="senz3d_depth_optical_joint" type="fixed">
+    <origin xyz="0.0 0.0 0.0" rpy="0.0 0.0 ${M_PI}" />
+    <parent link="senz3d_depth_frame"/>
+    <child link="senz3d_depth_optical_frame"/>
+  </joint>
+  <link name="senz3d_depth_optical_frame"/>
   <!-- Sonar links forming a half ring centered on (and slightly above) base_link-->
   <joint name="s_m90_joint" type="fixed">

Commit message: Camera description moved to the softkinetic repository: https://github.com/corot/softkinetic/commit/f8373d7618d79744d147eee2cee5c45870be6290

File: thorp_bringup/urdf/thorp.urdf.xacro (robot description, xacro)
@@ -14,9 +14,10 @@
   <xacro:include filename="$(find turtlebot_description)/urdf/turtlebot_library.urdf.xacro"/>
   <xacro:include filename="$(find turtlebot_arm_description)/urdf/arm.xacro"/>
+  <xacro:include filename="$(find softkinetic_camera)/urdf/senz3d.urdf.xacro"/>
   <!-- Plain Turtlebot 2 -->
   <kobuki/>
   <stack_hexagons parent="base_link"/>
   <sensor_kinect  parent="base_link"/>
-  <!-- Turtlebot arm plus mounting on Thorp -->
+  <!-- Turtlebot arm, its controller board and its mounting on Thorp -->
   <!-- Note that the arm position is biased to the left of the robot, and the dead angle also
        points to the left; with this configuration, the arm can reach most of the top plate -->
@@ -32,5 +33,5 @@
   <stack_bottom_pole parent="arm_base_link" number="12" x_loc="-0.038" y_loc="-0.0288" z_loc="-0.0112"/>
   <stack_bottom_pole parent="arm_base_link" number="13" x_loc="-0.038" y_loc=" 0.0288" z_loc="-0.0112"/>
-  <!-- Emulate the OpenCM9.04 as a box -->
+  <!-- Emulate the OpenCM9.04 controller as a box -->
   <joint name="opencm_joint" type="fixed">
     <origin xyz="0.045 0.03 0.008" rpy="0.0 0.0 0.0"/>
@@ -99,58 +100,11 @@
     </inertial>
   </link>
-  <!-- Camera -->
-  <joint name="senz3d_camera_joint" type="fixed">
-    <!-- <origin xyz="-0.045 -0.062 0.345" rpy="${M_PI/2 + 0.907571211037} 0.0 ${M_PI/2}"/> -->
+  <!-- The camera itself -->
+  <sensor_senz3d parent="plate_top_link" name="senz3d_camera">
+    <!-- Extrinsic parameters obtained through arm-camera calibration:
+         http://wiki.ros.org/turtlebot_arm_kinect_calibration -->
     <origin xyz="-0.0552702 -0.0411472 0.323393" rpy="2.3447 0.0160734 1.59265"/>
-    <parent link="plate_top_link"/>
-    <child link="senz3d_camera_link"/>
-  </joint>
-  <link name="senz3d_camera_link">
-    <visual>
-      <origin xyz="0.0 0.0 0.0" rpy="0.0 0.0 0.0"/>
-      <geometry>
-        <!-- As we don't have a Senz3D mesh, use a deformed Asus Xtion Pro instead -->
-        <mesh filename="package://turtlebot_description/meshes/sensors/asus_xtion_pro_live.dae" scale="0.0006 0.0015 0.001"/>
-      </geometry>
-    </visual>
-    <collision>
-      <origin xyz="0.0 0.0 -0.005" rpy="0 0 0"/>
-      <geometry>
-      <box size="0.11 0.04 0.04"/>
-    </geometry>
-    </collision>
-    <inertial>
-      <mass value="0.271"/>
-      <origin xyz="0 0 0"/>
-      <inertia ixx="0.001" ixy="0.0" ixz="0.0"
-        iyy="0.001" iyz="0.0"
-        izz="0.001"/>
-    </inertial>
-  </link>
-  <!-- Add frames for RGB and depth optical axes -->
-  <joint name="senz3d_rgb_joint" type="fixed">
-    <origin xyz="0.0125 0.0 0.0" rpy="0.0 0.0 0.0"/>
-    <parent link="senz3d_camera_link"/>
-    <child link="senz3d_rgb_frame"/>
-  </joint>
-  <link name="senz3d_rgb_frame"/>
-  <joint name="senz3d_rgb_optical_joint" type="fixed">
-    <origin xyz="0.0 0.0 0.0" rpy="0.0 0.0 ${M_PI}" />
-    <parent link="senz3d_rgb_frame"/>
-    <child link="senz3d_rgb_optical_frame"/>
-  </joint>
-  <link name="senz3d_rgb_optical_frame"/>
-  <joint name="senz3d_depth_joint" type="fixed">
-    <origin xyz="-0.0125 0.0 0.0" rpy="0.0 0.0 0.0"/>
-    <parent link="senz3d_camera_link"/>
-    <child link="senz3d_depth_frame"/>
-  </joint>
-  <link name="senz3d_depth_frame"/>
-  <joint name="senz3d_depth_optical_joint" type="fixed">
-    <origin xyz="0.0 0.0 0.0" rpy="0.0 0.0 ${M_PI}" />
-    <parent link="senz3d_depth_frame"/>
-    <child link="senz3d_depth_optical_frame"/>
-  </joint>
-  <link name="senz3d_depth_optical_frame"/>
+  </sensor_senz3d>
+  <!-- Additional frames for range sensors -->
   <!-- Sonar links forming a half ring centered on (and slightly above) base_link-->
   <joint name="s_m90_joint" type="fixed">

Commit message: Add a frame and KF to the arm IR sensor. I have also fixed the voltage-to-range calibration

File: thorp_bringup/urdf/thorp.urdf.xacro (robot description, xacro)
@@ -63,4 +63,11 @@
     </inertial>
   </link>
+  <!-- Arm IR sensor link, mounted below the arm mount and pointing forward -->
+  <joint name="ir_arm_joint" type="fixed">
+    <origin xyz="0.02  0.0 0.01" rpy="0.0 0.0 0.0"/>
+    <parent link="arm_base_link"/>
+    <child link="ir_arm_link"/>
+  </joint>
+  <link name="ir_arm_link"/>
   <!-- Senz3D camera plus mounting on Thorp -->
   <!-- Mounting poles: we emulate one top and two middle poles overlapping two top poles -->
