Commit message: As the calibration process assumes we use a kinect, and provides as output the tf from fixed frame to camera_link instead of to rgb_frame, we must "emulate" the kinect's tf scheme by reversing the camera_link -> rgb_frame tf and add the Senz3D camera_link -> rgb_frame

File: thorp_bringup/urdf/thorp.urdf.xacro (robot description, xacro)
@@ -24,5 +24,5 @@
   <turtlebot_arm parent="plate_top_link" color="white" gripper_color="black"
                  joints_vlimit="0.3571" pan_llimit="-4.189" pan_ulimit="1.047">
-    <origin xyz="0.11214 0.0295 0.0284"/>
+    <origin xyz="0.10914 0.0295 0.0284"/>
   </turtlebot_arm>
   <arm_mount parent="arm_base_link" name="arm_mount" color="black">
@@ -35,5 +35,5 @@
   <!-- Emulate the OpenCM9.04 controller as a box -->
   <joint name="opencm_joint" type="fixed">
-    <origin xyz="0.045 0.03 0.008" rpy="0.0 0.0 0.0"/>
+    <origin xyz="0.042 0.03 0.008" rpy="0.0 0.0 0.0"/>
     <parent link="plate_top_link"/>
     <child link="opencm_joint_link"/>
@@ -108,8 +108,24 @@
   </link>
   <!-- The camera itself -->
-  <sensor_senz3d parent="plate_top_link" name="senz3d_camera">
+  <joint name="senz3d_calib_joint" type="fixed">
     <!-- Extrinsic parameters obtained through arm-camera calibration:
          http://wiki.ros.org/turtlebot_arm_kinect_calibration -->
     <origin xyz="-0.0552702 -0.0411472 0.323393" rpy="2.3447 0.0160734 1.59265"/>
+    <parent link="plate_top_link"/>
+    <child link="senz3d_calib_link"/>
+  </joint>
+  <link name="senz3d_calib_link"/>
+  <!-- As the calibration process assumes we use a kinect, and provides as output the tf from fixed frame
+       to camera_link instead of to rgb_frame, we must "emulate" the kinect's tf scheme by reversing the
+       camera_link -> rgb_frame tf and add the Senz3D camera_link -> rgb_frame:
+        > Kinect camera_rgb_frame -> camera_link
+            -0.031, 0.013, -0.016, 0.000, 0.000, 0.000
+        > Rotate PI/2, 0.0, PI/2 to adapt to Senz3D frames
+             0.013, -0.016, -0.031, 0.000, 0.000, 0.000
+        > Remove Senz3D's camera_link -> rgb_frame tf (0.0125 on x-axis)
+             0.0005, -0.016, -0.031, 0.000, 0.000, 0.000
+    -->
+  <sensor_senz3d parent="senz3d_calib_link" name="senz3d_camera">
+    <origin xyz="0.0005 -0.016 -0.031" rpy="0.0 0.0 0.0"/>
   </sensor_senz3d>
   <!-- Additional frames for range sensors -->

Commit message: Replace calibration by camera base -> camera
Also added commented playing around with an external kinect

File: thorp_bringup/urdf/thorp.urdf.xacro (robot description, xacro)
@@ -19,4 +19,19 @@
   <stack_hexagons parent="base_link"/>
   <sensor_kinect  parent="base_link"/>
+<!--  playing around with an external kinect
+  <sensor_kinect  parent="fixed_external_camera_link"/>
+  <joint name="external_camera_joint" type="fixed">
+    <origin xyz="-0.117707 -0.732153 1.1196" rpy="-0.0205534 0.499254 0.901111"/>
+    <parent link="base_link"/>
+    <child link="external_camera_link"/>
+  </joint>
+  <link name="external_camera_link"/>
+  <joint name="fixed_external_camera_joint" type="fixed">
+    <origin xyz="0.0 -0.0125 0.025" rpy="0.0 0.0 0.0"/>
+    <parent link="external_camera_link"/>
+    <child link="fixed_external_camera_link"/>
+  </joint>
+  <link name="fixed_external_camera_link"/>
+-->
   <!-- Turtlebot arm, its controller board and its mounting on Thorp -->
   <!-- Note that the arm position is biased to the left of the robot, and the dead angle also
@@ -111,21 +126,11 @@
     <!-- Extrinsic parameters obtained through arm-camera calibration:
          http://wiki.ros.org/turtlebot_arm_kinect_calibration -->
-    <origin xyz="-0.0552702 -0.0411472 0.323393" rpy="2.3447 0.0160734 1.59265"/>
-    <parent link="plate_top_link"/>
+    <origin xyz="0.0236345 -0.035567 0.0125611" rpy="2.36437 0.0326246 1.55928"/>
+    <parent link="senz3d_mount_link"/>
     <child link="senz3d_calib_link"/>
   </joint>
   <link name="senz3d_calib_link"/>
-  <!-- As the calibration process assumes we use a kinect, and provides as output the tf from fixed frame
-       to camera_link instead of to rgb_frame, we must "emulate" the kinect's tf scheme by reversing the
-       camera_link -> rgb_frame tf and add the Senz3D camera_link -> rgb_frame:
-        > Kinect camera_rgb_frame -> camera_link
-            -0.031, 0.013, -0.016, 0.000, 0.000, 0.000
-        > Rotate PI/2, 0.0, PI/2 to adapt to Senz3D frames
-             0.013, -0.016, -0.031, 0.000, 0.000, 0.000
-        > Remove Senz3D's camera_link -> rgb_frame tf (0.0125 on x-axis)
-             0.0005, -0.016, -0.031, 0.000, 0.000, 0.000
-    -->
   <sensor_senz3d parent="senz3d_calib_link" name="senz3d_camera">
-    <origin xyz="0.0005 -0.016 -0.031" rpy="0.0 0.0 0.0"/>
+    <origin xyz="0.0 0.0 0.0" rpy="0.0 0.0 0.0"/>
   </sensor_senz3d>
   <!-- Additional frames for range sensors -->

Commit message: Add Gazebo support (work on progress)

File: thorp_bringup/urdf/thorp.urdf.xacro (robot description, xacro)
@@ -14,4 +14,5 @@
   <xacro:include filename="$(find turtlebot_description)/urdf/turtlebot_library.urdf.xacro"/>
   <xacro:include filename="$(find turtlebot_arm_description)/urdf/arm.xacro"/>
+  <xacro:include filename="$(find thorp_bringup)/urdf/thorp_gazebo.urdf.xacro"/>
   <xacro:include filename="$(find softkinetic_camera)/urdf/senz3d.urdf.xacro"/>
   <!-- Plain Turtlebot 2 -->
@@ -37,9 +38,9 @@
   <!-- Note that the arm position is biased to the left of the robot, and the dead angle also
        points to the left; with this configuration, the arm can reach most of the top plate -->
-  <turtlebot_arm parent="plate_top_link" color="white" gripper_color="black"
+  <turtlebot_arm parent="plate_top_link" color="White" gripper_color="Black"
                  joints_vlimit="0.3571" pan_llimit="-4.189" pan_ulimit="1.047">
     <origin xyz="0.10914 0.0295 0.0284"/>
   </turtlebot_arm>
-  <arm_mount parent="arm_base_link" name="arm_mount" color="black">
+  <arm_mount parent="arm_base_link" name="arm_mount" color="Black">
     <origin xyz="0.0 0.0 0.0" rpy="0.0 0.0 0.0"/>
   </arm_mount>
@@ -74,6 +75,6 @@
       <origin xyz="0 0 0"/>
       <inertia ixx="0.001" ixy="0.0" ixz="0.0"
-        iyy="0.001" iyz="0.0"
-        izz="0.001"/>
+               iyy="0.001" iyz="0.0"
+               izz="0.001"/>
     </inertial>
   </link>
@@ -104,5 +105,5 @@
         <box size="0.02 0.24 0.006"/>
       </geometry>
-      <material name="black">
+      <material name="Black">
         <color rgba="0.0 0.0 0.0 1.0"/>
       </material>
@@ -115,9 +116,9 @@
     </collision>
     <inertial>
-      <mass value="0.01"/>
+      <mass value="0.04"/>
       <origin xyz="0 0 0"/>
       <inertia ixx="0.001" ixy="0.0" ixz="0.0"
-        iyy="0.001" iyz="0.0"
-        izz="0.001"/>
+               iyy="0.001" iyz="0.0"
+               izz="0.001"/>
     </inertial>
   </link>

Commit message: Replicate kinect tf scheme. I should re-calibrate to validate my changes...

File: thorp_bringup/urdf/thorp.urdf.xacro (robot description, xacro)
@@ -127,5 +127,5 @@
     <!-- Extrinsic parameters obtained through arm-camera calibration:
          http://wiki.ros.org/turtlebot_arm_kinect_calibration -->
-    <origin xyz="0.0236345 -0.035567 0.0125611" rpy="2.36437 0.0326246 1.55928"/>
+    <origin xyz="0.0236345 -0.035567 0.0125611" rpy="0.0326246 ${2.36437 - M_PI/2} ${1.55928 - M_PI/2}"/>
     <parent link="senz3d_mount_link"/>
     <child link="senz3d_calib_link"/>

Commit message: Add gazebo simulation

File: thorp_bringup/urdf/thorp.urdf.xacro (robot description, xacro)
@@ -135,72 +135,44 @@
     <origin xyz="0.0 0.0 0.0" rpy="0.0 0.0 0.0"/>
   </sensor_senz3d>
-  <!-- Additional frames for range sensors -->
-  <!-- Sonar links forming a half ring centered on (and slightly above) base_link-->
-  <joint name="s_m90_joint" type="fixed">
-    <origin xyz="0.0     -0.15500 0.09" rpy="0.0 0.0 -1.57080"/>
-    <parent link="base_link"/>
-    <child link="s_m90_link"/>
-  </joint>
-  <link name="s_m90_link"/>
-  <joint name="s_m72_joint" type="fixed">
-    <origin xyz="0.04790 -0.14741 0.09" rpy="0.0 0.0 -1.25664"/>
-    <parent link="base_link"/>
-    <child link="s_m72_link"/>
-  </joint>
-  <link name="s_m72_link"/>
-  <joint name="s_m54_joint" type="fixed">
-    <origin xyz="0.09111 -0.12540 0.09" rpy="0.0 0.0 -0.94248"/>
-    <parent link="base_link"/>
-    <child link="s_m54_link"/>
-  </joint>
-  <link name="s_m54_link"/>
-  <joint name="s_m36_joint" type="fixed">
-    <origin xyz="0.12540 -0.09111 0.09" rpy="0.0 0.0 -0.62832"/>
-    <parent link="base_link"/>
-    <child link="s_m36_link"/>
-  </joint>
-  <link name="s_m36_link"/>
-  <joint name="s_m18_joint" type="fixed">
-    <origin xyz="0.14741 -0.04790 0.09" rpy="0.0 0.0 -0.31416"/>
-    <parent link="base_link"/>
-    <child link="s_m18_link"/>
-  </joint>
-  <link name="s_m18_link"/>
-  <joint name="s_0_joint" type="fixed">
-    <origin xyz="0.155    0.0     0.09" rpy="0.0 0.0 0.0"/>
-    <parent link="base_link"/>
-    <child link="s_0_link"/>
-  </joint>
-  <link name="s_0_link"/>
-  <joint name="s_p18_joint" type="fixed">
-    <origin xyz="0.14741  0.04790 0.09" rpy="0.0 0.0 0.31416"/>
-    <parent link="base_link"/>
-    <child link="s_p18_link"/>
-  </joint>
-  <link name="s_p18_link"/>
-  <joint name="s_p36_joint" type="fixed">
-    <origin xyz="0.12540  0.09111 0.09" rpy="0.0 0.0 0.62832"/>
-    <parent link="base_link"/>
-    <child link="s_p36_link"/>
-  </joint>
-  <link name="s_p36_link"/>
-  <joint name="s_p54_joint" type="fixed">
-    <origin xyz="0.09111  0.12540 0.09" rpy="0.0 0.0 0.94248"/>
-    <parent link="base_link"/>
-    <child link="s_p54_link"/>
-  </joint>
-  <link name="s_p54_link"/>
-  <joint name="s_p72_joint" type="fixed">
-    <origin xyz="0.04790  0.14741 0.09" rpy="0.0 0.0 1.25664"/>
-    <parent link="base_link"/>
-    <child link="s_p72_link"/>
-  </joint>
-  <link name="s_p72_link"/>
-  <joint name="s_p90_joint" type="fixed">
-    <origin xyz="0.0      0.155   0.09" rpy="0.0 0.0 1.57080"/>
-    <parent link="base_link"/>
-    <child link="s_p90_link"/>
-  </joint>
-  <link name="s_p90_link"/>
+  <!-- Sonar sensors forming a half ring centered on (and slightly above) base_link-->
+  <LV_MaxSonar_EZ2_sensor name="m90" parent="base_link" x_loc="0.0"     y_loc="-0.15500" yaw="-1.57080"/>
+  <LV_MaxSonar_EZ2_sensor name="m72" parent="base_link" x_loc="0.04790" y_loc="-0.14741" yaw="-1.25664"/>
+  <LV_MaxSonar_EZ2_sensor name="m54" parent="base_link" x_loc="0.09111" y_loc="-0.12540" yaw="-0.94248"/>
+  <LV_MaxSonar_EZ2_sensor name="m36" parent="base_link" x_loc="0.12540" y_loc="-0.09111" yaw="-0.62832"/>
+  <LV_MaxSonar_EZ2_sensor name="m18" parent="base_link" x_loc="0.14741" y_loc="-0.04790" yaw="-0.31416"/>
+  <LV_MaxSonar_EZ2_sensor name="0"   parent="base_link" x_loc="0.155"   y_loc=" 0.0"     yaw=" 0.0"/>
+  <LV_MaxSonar_EZ2_sensor name="p18" parent="base_link" x_loc="0.14741" y_loc="+0.04790" yaw="+0.31416"/>
+  <LV_MaxSonar_EZ2_sensor name="p36" parent="base_link" x_loc="0.12540" y_loc="+0.09111" yaw="+0.62832"/>
+  <LV_MaxSonar_EZ2_sensor name="p54" parent="base_link" x_loc="0.09111" y_loc="+0.12540" yaw="+0.94248"/>
+  <LV_MaxSonar_EZ2_sensor name="p72" parent="base_link" x_loc="0.04790" y_loc="+0.14741" yaw="+1.25664"/>
+  <LV_MaxSonar_EZ2_sensor name="p90" parent="base_link" x_loc="0.0"     y_loc="+0.15500" yaw="+1.57080"/>
+  <xacro:macro name="LV_MaxSonar_EZ2_sensor" params="name parent x_loc y_loc yaw">
+    <joint name="s_${name}_joint" type="fixed">
+      <origin xyz="${x_loc} ${y_loc} 0.105" rpy="0.0 0.0 ${yaw}"/>
+      <parent link="${parent}"/>
+      <child link="s_${name}_link"/>
+    </joint>
+    <link name="s_${name}_link">
+      <inertial>
+        <mass value="0.001"/>
+        <origin xyz="0 0 0" rpy="0 0 0"/>
+        <inertia ixx="0.001" ixy="0.0" ixz="0.0"
+                 iyy="0.001" iyz="0.0"
+                 izz="0.001"/>
+      </inertial>
+      <visual>
+        <origin xyz="0 0 0" rpy="0 0 0" />
+        <geometry>
+          <mesh filename="package://hector_sensors_description/meshes/sonar_sensor/max_sonar_ez4.dae"/>
+        </geometry>
+      </visual>
+      <collision>
+        <origin xyz="0 0 0" rpy="0 0 0"/>
+        <geometry>
+          <box size="0.01 0.01 0.01"/>
+        </geometry>
+      </collision>
+    </link>
+  </xacro:macro>
   <!-- IR sensor links, pointing at -155, pi, pi and 155 degrees -->
   <joint name="ir_l155_joint" type="fixed">

File: thorp_bringup/urdf/thorp_gazebo.urdf.xacro (robot description, xacro)
@@ -2,5 +2,5 @@
 <robot name="thorp_gazebo" xmlns:xacro="http://ros.org/wiki/xacro">
   <!-- Simulated Creative Senz3d camera -->
-  <gazebo reference="senz3d_camera">
+  <gazebo reference="senz3d_camera_link">
     <sensor type="depth" name="senz3d">
       <always_on>true</always_on>
@@ -38,7 +38,8 @@
     </sensor>
   </gazebo>
-  <xacro:macro name="Sharp_GP2Y0A21_IR_sensor" params="name">
-    <gazebo reference="${name}_link">
-      <sensor type="ray" name="${name}">
+  <!-- LV-MaxSonar-EZ2 ultrasound sensors -->
+  <xacro:macro name="LV_MaxSonar_EZ2_sim" params="name">
+    <gazebo reference="s_${name}_link">
+      <sensor type="ray" name="s_${name}">
         <always_on>true</always_on>
         <update_rate>20</update_rate>
@@ -47,31 +48,91 @@
           <scan>
             <horizontal>
-              <samples>50</samples>
-              <resolution>1.0</resolution>
+              <samples>6</samples>
+              <resolution>1</resolution>
+              <min_angle>-0.3</min_angle>  <!-- -17 degree -->
+              <max_angle>+0.3</max_angle>  <!-- +17 degree -->
+            </horizontal>
+            <vertical>
+              <samples>6</samples>
+              <resolution>1</resolution>
+              <min_angle>-0.3</min_angle>  <!-- -17 degree -->
+              <max_angle>+0.3</max_angle>  <!-- +17 degree -->
+            </vertical>
+          </scan>
+          <range>
+            <min>0.1</min>
+            <max>6.0</max>
+            <resolution>0.01</resolution>
+          </range>
+          <noise>
+            <type>gaussian</type>
+            <mean>0.0</mean>
+            <stddev>0.08</stddev>
+          </noise>
+        </ray>
+        <plugin name="gazebo_ros_s_${name}_controller" filename="libhector_gazebo_ros_sonar.so">
+          <gaussianNoise>0.05</gaussianNoise>
+          <topicName>mobile_base/sensors/sonars/${name}</topicName>
+          <frameId>s_${name}_link</frameId>
+        </plugin>
+      </sensor>
+    </gazebo>
+  </xacro:macro>
+  <LV_MaxSonar_EZ2_sim name="m90"/>
+  <LV_MaxSonar_EZ2_sim name="m72"/>
+  <LV_MaxSonar_EZ2_sim name="m54"/>
+  <LV_MaxSonar_EZ2_sim name="m36"/>
+  <LV_MaxSonar_EZ2_sim name="m18"/>
+  <LV_MaxSonar_EZ2_sim name="0"/>
+  <LV_MaxSonar_EZ2_sim name="p18"/>
+  <LV_MaxSonar_EZ2_sim name="p36"/>
+  <LV_MaxSonar_EZ2_sim name="p54"/>
+  <LV_MaxSonar_EZ2_sim name="p72"/>
+  <LV_MaxSonar_EZ2_sim name="p90"/>
+  <!-- Sharp GP2Y0A21 IR sensors -->
+  <xacro:macro name="Sharp_GP2Y0A21_IR_sim" params="name">
+    <gazebo reference="ir_${name}_link">
+      <sensor type="ray" name="ir_${name}">
+        <always_on>true</always_on>
+        <update_rate>20</update_rate>
+        <visualize>true</visualize>
+        <ray>
+          <scan>
+            <horizontal>
+              <samples>1</samples>
+              <resolution>1</resolution>
               <min_angle>-0.0436</min_angle>  <!-- -2.5 degree -->
-              <max_angle>0.0436</max_angle> <!-- 2.5 degree -->
+              <max_angle>+0.0436</max_angle>  <!-- +2.5 degree -->
             </horizontal>
-<!--            Can't use vertical rays until this bug is resolved: -->
-<!--            https://bitbucket.org/osrf/gazebo/issue/509/vertical-sensor-doesnt-works -->
-<!--            <vertical> -->
-<!--              <samples>50</samples> -->
-<!--              <resolution>1.0</resolution> -->
-<!--              <min_angle>-0.0436</min_angle>  -2.5 degree -->
-<!--              <max_angle>0.0436</max_angle> 2.5 degree -->
-<!--            </vertical> -->
+            <vertical>
+              <samples>1</samples>
+              <resolution>1</resolution>
+              <min_angle>-0.0436</min_angle>  <!-- -2.5 degree -->
+              <max_angle>+0.0436</max_angle>  <!-- +2.5 degree -->
+            </vertical>
           </scan>
           <range>
             <min>0.01</min>
             <max>0.80</max>
-            <resolution>1.0</resolution>
+            <resolution>0.01</resolution>
           </range>
+          <noise>
+            <type>gaussian</type>
+            <mean>0.0</mean>
+            <stddev>0.02</stddev>
+          </noise>
         </ray>
+        <plugin name="gazebo_ros_ir_${name}_controller" filename="libhector_gazebo_ros_sonar.so">
+          <gaussianNoise>0.005</gaussianNoise>
+          <topicName>mobile_base/sensors/infrared/${name}</topicName>
+          <frameId>ir_${name}_link</frameId>
+        </plugin>
       </sensor>
     </gazebo>
   </xacro:macro>
-  <Sharp_GP2Y0A21_IR_sensor name="ir_l155"/>
-  <Sharp_GP2Y0A21_IR_sensor name="ir_l180"/>
-  <Sharp_GP2Y0A21_IR_sensor name="ir_r180"/>
-  <Sharp_GP2Y0A21_IR_sensor name="ir_r155"/>
+  <Sharp_GP2Y0A21_IR_sim name="l155"/>
+  <Sharp_GP2Y0A21_IR_sim name="l180"/>
+  <Sharp_GP2Y0A21_IR_sim name="r180"/>
+  <Sharp_GP2Y0A21_IR_sim name="r155"/>
   <!-- Gazebo configuration for other structural parts -->
   <gazebo reference="senz3d_mount_link">
@@ -81,5 +142,5 @@
   </gazebo>
   <gazebo reference="opencm_joint_link">
-    <material>Gazebo/Green</material>
+    <material>Gazebo/Black</material>
     <selfCollide>true</selfCollide>
     <gravity>true</gravity>

Commit message: Recalibration forced by the the tf system change on senz3D camera

File: thorp_bringup/urdf/thorp.urdf.xacro (robot description, xacro)
@@ -6,6 +6,6 @@
     - 3d Sensor : kinect
   Thorp addons
-    - 11 sonar links
-    - 4 IR sensor links
+    - 11 sonars
+    - 5 IR sensors
     - Turtlebot arm
     - Senz3D camera
@@ -20,19 +20,4 @@
   <stack_hexagons parent="base_link"/>
   <sensor_kinect  parent="base_link"/>
-<!--  playing around with an external kinect
-  <sensor_kinect  parent="fixed_external_camera_link"/>
-  <joint name="external_camera_joint" type="fixed">
-    <origin xyz="-0.117707 -0.732153 1.1196" rpy="-0.0205534 0.499254 0.901111"/>
-    <parent link="base_link"/>
-    <child link="external_camera_link"/>
-  </joint>
-  <link name="external_camera_link"/>
-  <joint name="fixed_external_camera_joint" type="fixed">
-    <origin xyz="0.0 -0.0125 0.025" rpy="0.0 0.0 0.0"/>
-    <parent link="external_camera_link"/>
-    <child link="fixed_external_camera_link"/>
-  </joint>
-  <link name="fixed_external_camera_link"/>
--->
   <!-- Turtlebot arm, its controller board and its mounting on Thorp -->
   <!-- Note that the arm position is biased to the left of the robot, and the dead angle also
@@ -127,5 +112,5 @@
     <!-- Extrinsic parameters obtained through arm-camera calibration:
          http://wiki.ros.org/turtlebot_arm_kinect_calibration -->
-    <origin xyz="0.0236345 -0.035567 0.0125611" rpy="0.0326246 ${2.36437 - M_PI/2} ${1.55928 - M_PI/2}"/>
+    <origin xyz="0.0256095 -0.0275026 0.00772833" rpy="-0.0703076 0.788321 -0.0731844"/>
     <parent link="senz3d_mount_link"/>
     <child link="senz3d_calib_link"/>
