Commit message: Add sonar mount mesh

File: thorp_bringup/urdf/thorp.urdf.xacro (robot description, xacro)
@@ -38,7 +38,7 @@
     <origin xyz="0.042 0.03 0.008" rpy="0.0 0.0 0.0"/>
     <parent link="plate_top_link"/>
-    <child link="opencm_joint_link"/>
-  </joint>
-  <link name="opencm_joint_link">
+    <child link="opencm_link"/>
+  </joint>
+  <link name="opencm_link">
     <visual>
       <origin xyz="0.0 0.0 0.0" rpy="0.0 0.0 0.0"/>
@@ -120,19 +120,46 @@
     <origin xyz="0.0 0.0 0.0" rpy="0.0 0.0 0.0"/>
   </sensor_senz3d>
-  <!-- Sonar sensors forming a half ring centered on (and slightly above) base_link-->
-  <LV_MaxSonar_EZ2_sensor name="m90" parent="base_link" x_loc="0.0"     y_loc="-0.15500" yaw="-1.57080"/>
-  <LV_MaxSonar_EZ2_sensor name="m72" parent="base_link" x_loc="0.04790" y_loc="-0.14741" yaw="-1.25664"/>
-  <LV_MaxSonar_EZ2_sensor name="m54" parent="base_link" x_loc="0.09111" y_loc="-0.12540" yaw="-0.94248"/>
-  <LV_MaxSonar_EZ2_sensor name="m36" parent="base_link" x_loc="0.12540" y_loc="-0.09111" yaw="-0.62832"/>
-  <LV_MaxSonar_EZ2_sensor name="m18" parent="base_link" x_loc="0.14741" y_loc="-0.04790" yaw="-0.31416"/>
-  <LV_MaxSonar_EZ2_sensor name="0"   parent="base_link" x_loc="0.155"   y_loc=" 0.0"     yaw=" 0.0"/>
-  <LV_MaxSonar_EZ2_sensor name="p18" parent="base_link" x_loc="0.14741" y_loc="+0.04790" yaw="+0.31416"/>
-  <LV_MaxSonar_EZ2_sensor name="p36" parent="base_link" x_loc="0.12540" y_loc="+0.09111" yaw="+0.62832"/>
-  <LV_MaxSonar_EZ2_sensor name="p54" parent="base_link" x_loc="0.09111" y_loc="+0.12540" yaw="+0.94248"/>
-  <LV_MaxSonar_EZ2_sensor name="p72" parent="base_link" x_loc="0.04790" y_loc="+0.14741" yaw="+1.25664"/>
-  <LV_MaxSonar_EZ2_sensor name="p90" parent="base_link" x_loc="0.0"     y_loc="+0.15500" yaw="+1.57080"/>
+  <!-- Sonar sensors forming a half ring centered on (and slightly above) base_link -->
+  <joint name="sonars_joint" type="fixed">
+    <origin xyz="0.0 0.0 0.108" rpy="0.0 0.0 0.0"/>
+    <parent link="base_link"/>
+    <child link="sonars_mount_link"/>
+  </joint>
+  <link name="sonars_mount_link">
+    <inertial>
+      <mass value="0.22"/>
+      <origin xyz="0 0 0"/>
+      <inertia ixx="1.0" ixy="0.0" ixz="0.0"
+               iyy="1.0" iyz="0.0"
+               izz="1.0"/>
+    </inertial>
+    <visual>
+      <origin xyz="0.0 0.0 -0.058" rpy="${-M_PI/2} -${M_PI} ${-M_PI/2}"/>
+      <geometry>
+        <mesh filename="package://thorp_bringup/resources/meshes/sonar_array.stl" scale="0.001 0.001 0.001"/>
+      </geometry>
+      <material name="Black"/>
+    </visual>
+    <collision>
+      <origin xyz="-0.01 0.0 0.0165" rpy="0.0 0.0 0.0"/>
+      <geometry>
+        <box size="0.074 0.074 0.004"/>
+      </geometry>
+    </collision>
+  </link>
+  <LV_MaxSonar_EZ2_sensor name="m90" parent="sonars_mount_link" x_loc="0.0"    y_loc="-0.1380" yaw="-1.57080"/>
+  <LV_MaxSonar_EZ2_sensor name="m72" parent="sonars_mount_link" x_loc="0.0426" y_loc="-0.1312" yaw="-1.25664"/>
+  <LV_MaxSonar_EZ2_sensor name="m54" parent="sonars_mount_link" x_loc="0.0811" y_loc="-0.1116" yaw="-0.94248"/>
+  <LV_MaxSonar_EZ2_sensor name="m36" parent="sonars_mount_link" x_loc="0.1116" y_loc="-0.0811" yaw="-0.62832"/>
+  <LV_MaxSonar_EZ2_sensor name="m18" parent="sonars_mount_link" x_loc="0.1312" y_loc="-0.0426" yaw="-0.31416"/>
+  <LV_MaxSonar_EZ2_sensor name="0"   parent="sonars_mount_link" x_loc="0.138"  y_loc=" 0.0"    yaw=" 0.0"/>
+  <LV_MaxSonar_EZ2_sensor name="p18" parent="sonars_mount_link" x_loc="0.1312" y_loc="+0.0426" yaw="+0.31416"/>
+  <LV_MaxSonar_EZ2_sensor name="p36" parent="sonars_mount_link" x_loc="0.1116" y_loc="+0.0811" yaw="+0.62832"/>
+  <LV_MaxSonar_EZ2_sensor name="p54" parent="sonars_mount_link" x_loc="0.0811" y_loc="+0.1116" yaw="+0.94248"/>
+  <LV_MaxSonar_EZ2_sensor name="p72" parent="sonars_mount_link" x_loc="0.0426" y_loc="+0.1312" yaw="+1.25664"/>
+  <LV_MaxSonar_EZ2_sensor name="p90" parent="sonars_mount_link" x_loc="0.0"    y_loc="+0.1380" yaw="+1.57080"/>
   <xacro:macro name="LV_MaxSonar_EZ2_sensor" params="name parent x_loc y_loc yaw">
     <joint name="s_${name}_joint" type="fixed">
-      <origin xyz="${x_loc} ${y_loc} 0.105" rpy="0.0 0.0 ${yaw}"/>
+      <origin xyz="${x_loc} ${y_loc} 0.0" rpy="0.0 0.0 ${yaw}"/>
       <parent link="${parent}"/>
       <child link="s_${name}_link"/>

Commit message: Provide meaningful values for links' moment of inertia, but just epsilon values. The right formulas are explained here: http://en.wikipedia.org/wiki/List_of_moments_of_inertia

File: thorp_bringup/urdf/thorp.urdf.xacro (robot description, xacro)
@@ -59,7 +59,7 @@
       <mass value="0.01"/>
       <origin xyz="0 0 0"/>
-      <inertia ixx="0.001" ixy="0.0" ixz="0.0"
-               iyy="0.001" iyz="0.0"
-               izz="0.001"/>
+      <inertia ixx="0.0001" ixy="0.0" ixz="0.0"
+               iyy="0.0001" iyz="0.0"
+               izz="0.0001"/>
     </inertial>
   </link>
@@ -101,9 +101,9 @@
     </collision>
     <inertial>
-      <mass value="0.04"/>
+      <mass value="0.040"/>
       <origin xyz="0 0 0"/>
-      <inertia ixx="0.001" ixy="0.0" ixz="0.0"
-               iyy="0.001" iyz="0.0"
-               izz="0.001"/>
+      <inertia ixx="0.0001" ixy="0.0" ixz="0.0"
+               iyy="0.0001" iyz="0.0"
+               izz="0.0001"/>
     </inertial>
   </link>
@@ -130,7 +130,7 @@
       <mass value="0.22"/>
       <origin xyz="0 0 0"/>
-      <inertia ixx="1.0" ixy="0.0" ixz="0.0"
-               iyy="1.0" iyz="0.0"
-               izz="1.0"/>
+      <inertia ixx="0.0001" ixy="0.0" ixz="0.0"
+               iyy="0.0001" iyz="0.0"
+               izz="0.0001"/>
     </inertial>
     <visual>
@@ -169,7 +169,7 @@
         <mass value="0.001"/>
         <origin xyz="0 0 0" rpy="0 0 0"/>
-        <inertia ixx="0.001" ixy="0.0" ixz="0.0"
-                 iyy="0.001" iyz="0.0"
-                 izz="0.001"/>
+        <inertia ixx="0.000001" ixy="0.0" ixz="0.0"
+                 iyy="0.000001" iyz="0.0"
+                 izz="0.000001"/>
       </inertial>
       <visual>

Commit message: Pass a "simulation" parameter to the xacro robot desciption so we can use "ideal" values for camera pose instead of the ones obtained from calibration. **WARNING:** this will create problems whe running the whole physical robot, as turtlebot_bringup minimal.launch also launches a robot_state_publisher

File: thorp_bringup/urdf/thorp.urdf.xacro (robot description, xacro)
@@ -112,5 +112,10 @@
     <!-- Extrinsic parameters obtained through arm-camera calibration:
          http://wiki.ros.org/turtlebot_arm_kinect_calibration -->
-    <origin xyz="0.0256095 -0.0275026 0.00772833" rpy="-0.0703076 0.788321 -0.0731844"/>
+    <xacro:if value="$(arg simulation)">
+      <origin xyz="0.0256095 -0.0275026 0.00772833" rpy="0.0 0.788321 0.0"/>
+    </xacro:if>
+    <xacro:unless value="$(arg simulation)">
+      <origin xyz="0.0256095 -0.0275026 0.00772833" rpy="-0.0703076 0.788321 -0.0731844"/>
+    </xacro:unless>
     <parent link="senz3d_mount_link"/>
     <child link="senz3d_calib_link"/>

Commit message: Seems like Gazebo kinect plugin needs to use a centered frame instead of separated rgb and depth

File: thorp_bringup/urdf/thorp.urdf.xacro (robot description, xacro)
@@ -132,4 +132,14 @@
   </joint>
   <link name="senz3d_calib_link"/>
+  <!-- Seems like Gazebo kinect plugin needs to use a centered frame instead of separated rgb and depth.
+       No idea if this makes any sense, but it works! -->
+  <xacro:if value="$(arg simulation)">
+    <joint name="senz3d_camera_gazebo_optical_joint" type="fixed">
+      <origin xyz="0.0 0.0 0.0" rpy="${-M_PI/2} 0.0 ${-M_PI/2}"/>
+      <parent link="senz3d_camera_link"/>
+      <child link="senz3d_camera_gazebo_optical_frame"/>
+    </joint>
+    <link name="senz3d_camera_gazebo_optical_frame"/>
+  </xacro:if>
   <sensor_senz3d parent="senz3d_calib_link" name="senz3d_camera">
     <origin xyz="0.0 0.0 0.0" rpy="0.0 0.0 0.0"/>

File: thorp_bringup/urdf/thorp_gazebo.urdf.xacro (robot description, xacro)
@@ -27,5 +27,5 @@
         <cameraInfoTopicName>rgb/camera_info</cameraInfoTopicName>
         <depthImageCameraInfoTopicName>depth/camera_info</depthImageCameraInfoTopicName>
-        <frameName>senz3d_camera_depth_optical_frame</frameName>
+        <frameName>senz3d_camera_gazebo_optical_frame</frameName>
         <baseline>0.1</baseline>
         <distortion_k1>0.0</distortion_k1>

Commit message: I also move the optical tf a bit forward to make pointcloud match better the model; this is absolutely arbitrary

File: thorp_bringup/urdf/thorp.urdf.xacro (robot description, xacro)
@@ -133,8 +133,9 @@
   <link name="senz3d_calib_link"/>
   <!-- Seems like Gazebo kinect plugin needs to use a centered frame instead of separated rgb and depth.
-       No idea if this makes any sense, but it works! -->
+       No idea if this makes any sense, but it works! I also move the optical tf a bit forward to make
+       pointcloud match better the model; this is absolutely arbitrary... -->
   <xacro:if value="$(arg simulation)">
     <joint name="senz3d_camera_gazebo_optical_joint" type="fixed">
-      <origin xyz="0.0 0.0 0.0" rpy="${-M_PI/2} 0.0 ${-M_PI/2}"/>
+      <origin xyz="0.004 0.0 0.0" rpy="${-M_PI/2} 0.0 ${-M_PI/2}"/>
       <parent link="senz3d_camera_link"/>
       <child link="senz3d_camera_gazebo_optical_frame"/>

Commit message: Replace sonar ring mesh with a collada, as the stl somehow stopped working Also resize it and the sonars to avoid seeing ugly green and silver colors behind

File: thorp_bringup/urdf/thorp.urdf.xacro (robot description, xacro)
@@ -161,9 +161,8 @@
     </inertial>
     <visual>
-      <origin xyz="0.0 0.0 -0.058" rpy="${-M_PI/2} -${M_PI} ${-M_PI/2}"/>
-      <geometry>
-        <mesh filename="package://thorp_bringup/resources/meshes/sonar_array.stl" scale="0.001 0.001 0.001"/>
-      </geometry>
-      <material name="Black"/>
+      <origin xyz="0.0 0.0 -0.0586" rpy="${-M_PI/2} -${M_PI} ${-M_PI/2}"/>
+      <geometry>
+        <mesh filename="package://thorp_bringup/resources/meshes/sonar_array.dae" scale="0.001006 0.001006 0.001"/>
+      </geometry>
     </visual>
     <collision>
@@ -202,5 +201,5 @@
         <origin xyz="0 0 0" rpy="0 0 0" />
         <geometry>
-          <mesh filename="package://hector_sensors_description/meshes/sonar_sensor/max_sonar_ez4.dae"/>
+          <mesh filename="package://hector_sensors_description/meshes/sonar_sensor/max_sonar_ez4.dae" scale="1.1 1.1 1.1"/>/>
         </geometry>
       </visual>

Commit message: Use the STL model for Senz 3D mounting plate

File: thorp_bringup/urdf/thorp.urdf.xacro (robot description, xacro)
@@ -88,5 +88,5 @@
   <stack_top_pole parent="plate_top_link" number="12" x_loc="-0.0874" y_loc=" 0.098" z_loc="${0.006/2 + 0.2032/2 + 0.1}"/>
   <stack_top_pole parent="plate_top_link" number="13" x_loc="-0.0874" y_loc="-0.098" z_loc="${0.006/2 + 0.2032/2 + 0.1}"/>
-  <!-- Mounting plate; this structure is provisional -->
+  <!-- Mounting plate -->
   <joint name="senz3d_mount_joint" type="fixed">
     <origin xyz="-0.0874 0.0 ${0.2032 + 0.006 + 0.1}" rpy="0.0 0.0 0.0"/>
@@ -96,7 +96,7 @@
   <link name="senz3d_mount_link">
     <visual>
-      <origin xyz="0.0 0.0 0.0" rpy="0.0 0.0 0.0"/>
-      <geometry>
-        <box size="0.02 0.24 0.006"/>
+      <origin xyz="0.0075 0.0 -0.003" rpy="0.0 0.0 0.0"/>
+      <geometry>
+        <mesh filename="package://thorp_bringup/resources/meshes/senz3d_mount.stl" scale="0.001 0.001 0.001"/>
       </geometry>
       <material name="Black">
@@ -105,7 +105,7 @@
     </visual>
     <collision>
-      <origin xyz="0.0 0.0 0.0" rpy="0.0 0.0 0.0"/>
-      <geometry>
-        <box size="0.02 0.24 0.006"/>
+      <origin xyz="-0.0075 0.0 0.0" rpy="0.0 0.0 0.0"/>
+      <geometry>
+        <box size="0.03 0.22 0.006"/>
       </geometry>
     </collision>

Commit message: Updated camera position

File: thorp_bringup/urdf/thorp.urdf.xacro (robot description, xacro)
@@ -120,11 +120,12 @@
   <!-- The camera itself -->
   <joint name="senz3d_calib_joint" type="fixed">
+    <!-- Ideal extrinsic parameters obtained from robot model -->
+    <xacro:if value="$(arg simulation)">
+      <origin xyz="0.02 -0.03 0.022" rpy="0.0 0.65 0.0"/>
+    </xacro:if>
     <!-- Extrinsic parameters obtained through arm-camera calibration:
          http://wiki.ros.org/turtlebot_arm_kinect_calibration -->
-    <xacro:if value="$(arg simulation)">
-      <origin xyz="0.0256095 -0.0275026 0.00772833" rpy="0.0 0.788321 0.0"/>
-    </xacro:if>
     <xacro:unless value="$(arg simulation)">
-      <origin xyz="0.0256095 -0.0275026 0.00772833" rpy="-0.0703076 0.788321 -0.0731844"/>
+      <origin xyz="0.0285866 -0.03 0.0224632" rpy="-0.0488757 0.65176 -0.0463025"/>
     </xacro:unless>
     <parent link="senz3d_mount_link"/>

Commit message: Recalibrated... but still fails to grasp blocks in the right side!

File: thorp_bringup/urdf/thorp.urdf.xacro (robot description, xacro)
@@ -128,5 +128,7 @@
          http://wiki.ros.org/turtlebot_arm_kinect_calibration -->
     <xacro:unless value="$(arg simulation)">
-      <origin xyz="0.0285866 -0.03 0.0224632" rpy="-0.0488757 0.65176 -0.0463025"/>
+      <!-- <origin xyz="0.0277244 -0.0265666 0.0112677" rpy="-0.0328226 0.623228 -0.0172978"/> -->
+      <!-- <origin xyz="0.0273934 -0.015 0.0128054" rpy="-0.0502534 0.629487 -0.05"/> -->
+      <origin xyz="0.0305095 -0.0164463 0.0134078" rpy="-0.0369783 0.634554 -0.000672493"/>
     </xacro:unless>
     <parent link="senz3d_mount_link"/>

Commit message: Increase joints velocity limits for faster operation

File: thorp_bringup/urdf/thorp.urdf.xacro (robot description, xacro)
@@ -24,6 +24,7 @@
        is biased to the right; with this configuration, the arm lefts doesn't block completely
        camera view to the operation space.
-       We also use a deliberately low joints velocity limit to improve safety and precision -->
-  <xacro:property name="joints_vlimit" value="0.3571"/>
+       We also use a deliberately low joints velocity limit to improve safety and precision;
+       The phisical limit of the AX-12 is 114 rpm (684 deg/s) -->
+  <xacro:property name="joints_vlimit" value="0.8"/>
   <xacro:property name="pan_llimit" value="-2.617"/>
   <xacro:property name="pan_ulimit" value=" 2.617"/>

Commit message: Reduce elbow lower limit to force the arm to operate always with the same gripper orientation (and prevent the ridiculous full turns of the arm)

File: thorp_bringup/urdf/thorp.urdf.xacro (robot description, xacro)
@@ -31,5 +31,5 @@
   <xacro:property name="shoulder_llimit" value="-2.617"/>
   <xacro:property name="shoulder_ulimit" value=" 2.617"/>
-  <xacro:property name="elbow_llimit" value="-2.617"/>
+  <xacro:property name="elbow_llimit" value=" 0.0"/>
   <xacro:property name="elbow_ulimit" value=" 2.617"/>
   <xacro:property name="wrist_llimit" value="-1.745"/>

Commit message: Experiment: constrain the elbow lower limit and both shoulder limits to force the arm to operate always with the same gripper orientation, preventing the inefficient full turns. I don't think we need to be that restrictive, but it works fine now. We should anyway do a better problem assessment.

File: thorp_bringup/urdf/thorp.urdf.xacro (robot description, xacro)
@@ -24,9 +24,16 @@
        is biased to the right; with this configuration, the arm lefts doesn't block completely
        camera view to the operation space.
+       We constrain the elbow lower limit and both shoulder limits to force the arm to operate
+       always with the same gripper orientation, preventing the inefficient full turns.
+       TODO: I don't think we need to be that restrictive; do a better problem assessment.
        We also use a deliberately low joints velocity limit to improve safety and precision;
-       The phisical limit of the AX-12 is 114 rpm (684 deg/s) -->
+       The physical limit of the AX-12 is 114 rpm (684 deg/s) -->
   <xacro:property name="joints_vlimit" value="0.8"/>
+<!--
   <xacro:property name="pan_llimit" value="-2.617"/>
   <xacro:property name="pan_ulimit" value=" 2.617"/>
+ -->
+  <xacro:property name="pan_llimit" value="${-M_PI/2}"/>
+  <xacro:property name="pan_ulimit" value="${+M_PI/2}"/>
   <xacro:property name="shoulder_llimit" value="-2.617"/>
   <xacro:property name="shoulder_ulimit" value=" 2.617"/>
@@ -48,5 +55,5 @@
   <!-- Emulate the OpenCM9.04 controller as a box -->
   <joint name="opencm_joint" type="fixed">
-    <origin xyz="0.042 0.03 0.008" rpy="0.0 0.0 0.0"/>
+    <origin xyz="0.045 0.03 0.008" rpy="0.0 0.0 0.0"/>
     <parent link="plate_top_link"/>
     <child link="opencm_link"/>
