Commit message: Replace the Creative Senz3D by an Asus Xtion Pro, regenerating also the moveit configuration. As the Asus depth images are much less noisy, we can use now DepthImageOctomapUpdater instead of PointCloudOctomapUpdater to create the octomap, saving a ton of CPU.
TODO: try also on Gazebo simulation

File: thorp_bringup/urdf/thorp.urdf.xacro (robot description, xacro)
@@ -9,5 +9,5 @@
     - 5 IR sensors
     - Turtlebot arm
-    - Senz3D camera
+    - Manipulation 3d sensor (Asus Xtion Pro)
 -->
 <robot name="Thorp" xmlns:xacro="http://ros.org/wiki/xacro">
@@ -15,13 +15,15 @@
   <xacro:include filename="$(find turtlebot_arm_description)/urdf/turtlebot_arm.xacro"/>
   <xacro:include filename="$(find thorp_bringup)/urdf/thorp_gazebo.urdf.xacro"/>
-  <xacro:include filename="$(find softkinetic_camera)/urdf/senz3d.urdf.xacro"/>
+  <xacro:include filename="$(find thorp_bringup)/urdf/kinect.urdf.xacro"/>
+  <xacro:include filename="$(find thorp_bringup)/urdf/xtion.urdf.xacro"/>
+  <xacro:arg name="simulation" default="false"/>
   <!-- Plain Turtlebot 2 -->
   <kobuki/>
   <stack_hexagons parent="base_link"/>
-  <sensor_kinect  parent="base_link"/>
+  <kinect_camera parent="base_link" name="kinect"/>
   <!-- Turtlebot arm, its controller board and its mounting on Thorp -->
-  <!-- Note that the arm position is biased to the left of the robot, while the Senz3D camera
-       is biased to the right; with this configuration, the arm lefts doesn't block completely
-       camera view to the operation space.
+  <!-- Note that the arm position is biased to the left of the robot, while the manipulation
+       camera is biased to the right; with this configuration, the arm doesn't block completely
+       the camera vision of the operation space.
        We constrain the elbow lower limit and both shoulder limits to force the arm to operate
        always with the same gripper orientation, preventing the inefficient full turns.
@@ -90,31 +92,28 @@
   </joint>
   <link name="ir_arm_link"/>
-  <!-- Senz3D camera plus mounting on Thorp -->
-  <!-- Mounting poles: we emulate one top and two middle poles overlapping two top poles -->
-  <!-- The Z loc of the upper poles is : 1/2*plate height + 1/2*top pole height + 2*middle pole height (without screw) -->
-  <stack_top_pole parent="plate_top_link" number="10" x_loc="-0.0874" y_loc=" 0.098" z_loc="${0.006/2 + 0.2032/2}"/>
-  <stack_top_pole parent="plate_top_link" number="11" x_loc="-0.0874" y_loc="-0.098" z_loc="${0.006/2 + 0.2032/2}"/>
-  <stack_top_pole parent="plate_top_link" number="12" x_loc="-0.0874" y_loc=" 0.098" z_loc="${0.006/2 + 0.2032/2 + 0.1}"/>
-  <stack_top_pole parent="plate_top_link" number="13" x_loc="-0.0874" y_loc="-0.098" z_loc="${0.006/2 + 0.2032/2 + 0.1}"/>
+  <!-- Asus Xtion Pro camera plus mounting on Thorp -->
+  <!-- Mounting poles: two pairs of stacked top poles -->
+  <!-- The Z loc of the upper poles is : 1/2*plate height + 3/2*top pole height -->
+  <stack_top_pole parent="plate_top_link" number="10" x_loc="-0.0874" y_loc=" 0.098" z_loc="${0.006/2 + 0.2032*(1/2)}"/>
+  <stack_top_pole parent="plate_top_link" number="11" x_loc="-0.0874" y_loc="-0.098" z_loc="${0.006/2 + 0.2032*(1/2)}"/>
+  <stack_top_pole parent="plate_top_link" number="12" x_loc="-0.0874" y_loc=" 0.098" z_loc="${0.006/2 + 0.2032*(3/2)}"/>
+  <stack_top_pole parent="plate_top_link" number="13" x_loc="-0.0874" y_loc="-0.098" z_loc="${0.006/2 + 0.2032*(3/2)}"/>
   <!-- Mounting plate -->
-  <joint name="senz3d_mount_joint" type="fixed">
-    <origin xyz="-0.0874 0.0 ${0.2032 + 0.006 + 0.1}" rpy="0.0 0.0 0.0"/>
+  <joint name="xtion_mount_joint" type="fixed">
+    <origin xyz="-0.0874 0.0 ${0.2032*2 + 0.006}" rpy="0.0 ${M_PI/4} 0.0"/>
     <parent link="plate_top_link"/>
-    <child link="senz3d_mount_link"/>
-  </joint>
-  <link name="senz3d_mount_link">
+    <child link="xtion_mount_link"/>
+  </joint>
+  <link name="xtion_mount_link">
     <visual>
-      <origin xyz="0.0075 0.0 -0.003" rpy="0.0 0.0 0.0"/>
-      <geometry>
-        <mesh filename="package://thorp_bringup/resources/meshes/senz3d_mount.stl" scale="0.001 0.001 0.001"/>
-      </geometry>
-      <material name="Black">
-        <color rgba="0.0 0.0 0.0 1.0"/>
-      </material>
+      <origin xyz="0.0 0.0 0.0" rpy="${-M_PI/2} 0.0 0.0"/>
+      <geometry>
+        <mesh filename="package://turtlebot_description/meshes/sensors/xtion_pro_stack.dae"/>
+      </geometry>
     </visual>
     <collision>
-      <origin xyz="-0.0075 0.0 0.0" rpy="0.0 0.0 0.0"/>
-      <geometry>
-        <box size="0.03 0.22 0.006"/>
+      <origin xyz="0.0 0.0 0.0" rpy="0.0 0.0 0.0"/>
+      <geometry>
+        <box size="0.028 0.225 0.012"/>
       </geometry>
     </collision>
@@ -122,40 +121,33 @@
       <mass value="0.040"/>
       <origin xyz="0 0 0"/>
-      <inertia ixx="0.0001" ixy="0.0" ixz="0.0"
-               iyy="0.0001" iyz="0.0"
-               izz="0.0001"/>
+        <inertia ixx="0.0001" ixy="0.0" ixz="0.0"
+                 iyy="0.0001" iyz="0.0"
+                 izz="0.0001"/>
     </inertial>
   </link>
   <!-- The camera itself -->
-  <joint name="senz3d_calib_joint" type="fixed">
+  <xtion_camera parent="xtion_mount_link" name="xtion">
     <!-- Ideal extrinsic parameters obtained from robot model -->
     <xacro:if value="$(arg simulation)">
-      <origin xyz="0.02 -0.03 0.022" rpy="0.0 0.65 0.0"/>
+      <!-- <origin xyz="0.0 -0.025 0.015" rpy="0.0 0.0 0.0"/> -->
+      <origin xyz="0.015 0.01 0.015" rpy="0.0 0.0 0.0"/>
     </xacro:if>
     <!-- Extrinsic parameters obtained through arm-camera calibration:
          http://wiki.ros.org/turtlebot_arm_kinect_calibration -->
     <xacro:unless value="$(arg simulation)">
-      <!-- <origin xyz="0.0277244 -0.0265666 0.0112677" rpy="-0.0328226 0.623228 -0.0172978"/> -->
-      <!-- <origin xyz="0.0273934 -0.015 0.0128054" rpy="-0.0502534 0.629487 -0.05"/> -->
-      <origin xyz="0.0305095 -0.0164463 0.0134078" rpy="-0.0369783 0.634554 -0.000672493"/>
+      <origin xyz="0.015 0.01 0.015" rpy="0.0 0.0 0.0"/>
     </xacro:unless>
-    <parent link="senz3d_mount_link"/>
-    <child link="senz3d_calib_link"/>
-  </joint>
-  <link name="senz3d_calib_link"/>
+  </xtion_camera>
   <!-- Seems like Gazebo kinect plugin needs to use a centered frame instead of separated rgb and depth.
        No idea if this makes any sense, but it works! I also move the optical tf a bit forward to make
        pointcloud match better the model; this is absolutely arbitrary... -->
   <xacro:if value="$(arg simulation)">
-    <joint name="senz3d_camera_gazebo_optical_joint" type="fixed">
+    <joint name="xtion_gazebo_optical_joint" type="fixed">
       <origin xyz="0.004 0.0 0.0" rpy="${-M_PI/2} 0.0 ${-M_PI/2}"/>
-      <parent link="senz3d_camera_link"/>
-      <child link="senz3d_camera_gazebo_optical_frame"/>
+      <parent link="xtion_link"/>
+      <child link="xtion_gazebo_optical_frame"/>
     </joint>
-    <link name="senz3d_camera_gazebo_optical_frame"/>
+    <link name="xtion_gazebo_optical_frame"/>
   </xacro:if>
-  <sensor_senz3d parent="senz3d_calib_link" name="senz3d_camera">
-    <origin xyz="0.0 0.0 0.0" rpy="0.0 0.0 0.0"/>
-  </sensor_senz3d>
   <!-- Sonar sensors forming a half ring centered on (and slightly above) base_link -->
   <joint name="sonars_joint" type="fixed">

Commit message: Mount the Asus Xtion Pro raised and further back to increase covered manipulation area. I have also recovered the Senz3D in an intermediate position in the tower, but it is not used by now.

File: thorp_bringup/urdf/thorp.urdf.xacro (robot description, xacro)
@@ -4,14 +4,16 @@
     - Base      : kobuki
     - Stacks    : hexagons
-    - 3d Sensor : kinect
+    - 3D Sensor : kinect
   Thorp addons
     - 11 sonars
     - 5 IR sensors
     - Turtlebot arm
-    - Manipulation 3d sensor (Asus Xtion Pro)
+    - Auxiliary 3D sensor (Creative Senz3D)
+    - Manipulation 3D sensor (Asus Xtion Pro)
 -->
 <robot name="Thorp" xmlns:xacro="http://ros.org/wiki/xacro">
   <xacro:include filename="$(find turtlebot_description)/urdf/turtlebot_library.urdf.xacro"/>
   <xacro:include filename="$(find turtlebot_arm_description)/urdf/turtlebot_arm.xacro"/>
+  <xacro:include filename="$(find softkinetic_camera)/urdf/senz3d.urdf.xacro"/>
   <xacro:include filename="$(find thorp_bringup)/urdf/thorp_gazebo.urdf.xacro"/>
   <xacro:include filename="$(find thorp_bringup)/urdf/kinect.urdf.xacro"/>
@@ -92,28 +94,96 @@
   </joint>
   <link name="ir_arm_link"/>
-  <!-- Asus Xtion Pro camera plus mounting on Thorp -->
-  <!-- Mounting poles: two pairs of stacked top poles -->
+  <!-- Auxiliary Senz3D camera plus mounting on Thorp -->
+  <!-- Mounting poles: two columns made with one top and one middle poles stacked -->
+  <!-- The Z loc of the upper poles is : 1/2*plate height + top pole height + 1/2*middle pole height (without screw) -->
+  <stack_top_pole parent="plate_top_link" number="10" x_loc="-0.1124" y_loc=" 0.098" z_loc="${0.006/2 + 0.2032/2}"/>
+  <stack_top_pole parent="plate_top_link" number="20" x_loc="-0.1124" y_loc="-0.098" z_loc="${0.006/2 + 0.2032/2}"/>
+  <stack_middle_pole parent="plate_top_link" number="11" x_loc="-0.1124" y_loc=" 0.098" z_loc="${0.006/2 + 0.2032 + 0.0608/2}"/>
+  <stack_middle_pole parent="plate_top_link" number="21" x_loc="-0.1124" y_loc="-0.098" z_loc="${0.006/2 + 0.2032 + 0.0608/2}"/>
+  <!-- Mounting plate -->
+  <joint name="senz3d_mount_joint" type="fixed">
+    <origin xyz="-0.1124 0.0 ${0.2032 + 0.006 + 0.0515}" rpy="0.0 0.0 0.0"/>
+    <parent link="plate_top_link"/>
+    <child link="senz3d_mount_link"/>
+  </joint>
+  <link name="senz3d_mount_link">
+    <visual>
+      <origin xyz="0.0075 0.0 -0.003" rpy="0.0 0.0 0.0"/>
+      <geometry>
+        <mesh filename="package://thorp_bringup/resources/meshes/senz3d_mount.stl" scale="0.001 0.001 0.001"/>
+      </geometry>
+      <material name="Black">
+        <color rgba="0.0 0.0 0.0 1.0"/>
+      </material>
+    </visual>
+    <collision>
+      <origin xyz="-0.0075 0.0 0.0" rpy="0.0 0.0 0.0"/>
+      <geometry>
+        <box size="0.03 0.22 0.006"/>
+      </geometry>
+    </collision>
+    <inertial>
+      <mass value="0.040"/>
+      <origin xyz="0 0 0"/>
+      <inertia ixx="0.0001" ixy="0.0" ixz="0.0"
+               iyy="0.0001" iyz="0.0"
+               izz="0.0001"/>
+    </inertial>
+  </link>
+  <!-- The camera itself -->
+  <joint name="senz3d_calib_joint" type="fixed">
+    <!-- Ideal extrinsic parameters obtained from robot model -->
+    <xacro:if value="$(arg simulation)">
+      <origin xyz="0.02 0.013 0.022" rpy="0.0 0.0 0.0"/>
+    </xacro:if>
+    <!-- Extrinsic parameters obtained through arm-camera calibration:
+         http://wiki.ros.org/turtlebot_arm_kinect_calibration -->
+    <!-- NOTE: Not required by now in its role of auxiliary camera -->
+    <xacro:unless value="$(arg simulation)">
+      <origin xyz="0.02 0.013 0.022" rpy="0.0 0.0 0.0"/>
+    </xacro:unless>
+    <parent link="senz3d_mount_link"/>
+    <child link="senz3d_calib_link"/>
+  </joint>
+  <link name="senz3d_calib_link"/>
+  <!-- Seems like Gazebo kinect plugin needs to use a centered frame instead of separated rgb and depth.
+       No idea if this makes any sense, but it works! I also move the optical tf a bit forward to make
+       pointcloud match better the model; this is absolutely arbitrary... -->
+  <xacro:if value="$(arg simulation)">
+    <joint name="senz3d_gazebo_optical_joint" type="fixed">
+      <origin xyz="0.004 0.0 0.0" rpy="${-M_PI/2} 0.0 ${-M_PI/2}"/>
+      <parent link="senz3d_link"/>
+      <child link="senz3d_gazebo_optical_frame"/>
+    </joint>
+    <link name="senz3d_gazebo_optical_frame"/>
+  </xacro:if>
+  <sensor_senz3d parent="senz3d_calib_link" name="senz3d">
+    <origin xyz="0.0 0.0 0.0" rpy="0.0 0.0 0.0"/>
+  </sensor_senz3d>
+  <!-- Manipulation Asus Xtion Pro camera mounted on top of the Senz3D's mounting plate-->
+  <!-- Mounting poles: a pair of top poles -->
   <!-- The Z loc of the upper poles is : 1/2*plate height + 3/2*top pole height -->
-  <stack_top_pole parent="plate_top_link" number="10" x_loc="-0.0874" y_loc=" 0.098" z_loc="${0.006/2 + 0.2032*(1/2)}"/>
-  <stack_top_pole parent="plate_top_link" number="11" x_loc="-0.0874" y_loc="-0.098" z_loc="${0.006/2 + 0.2032*(1/2)}"/>
-  <stack_top_pole parent="plate_top_link" number="12" x_loc="-0.0874" y_loc=" 0.098" z_loc="${0.006/2 + 0.2032*(3/2)}"/>
-  <stack_top_pole parent="plate_top_link" number="13" x_loc="-0.0874" y_loc="-0.098" z_loc="${0.006/2 + 0.2032*(3/2)}"/>
+  <stack_top_pole parent="senz3d_mount_link" number="12" x_loc="0.0" y_loc=" 0.098" z_loc="${0.006/2 + 0.2032/2}"/>
+  <stack_top_pole parent="senz3d_mount_link" number="22" x_loc="0.0" y_loc="-0.098" z_loc="${0.006/2 + 0.2032/2}"/>
   <!-- Mounting plate -->
   <joint name="xtion_mount_joint" type="fixed">
-    <origin xyz="-0.0874 0.0 ${0.2032*2 + 0.006}" rpy="0.0 ${M_PI/4} 0.0"/>
-    <parent link="plate_top_link"/>
+    <origin xyz="0.0 0.0 ${0.2032 + 0.006}" rpy="0.0 0.0 0.0"/>
+    <parent link="senz3d_mount_link"/>
     <child link="xtion_mount_link"/>
   </joint>
   <link name="xtion_mount_link">
     <visual>
-      <origin xyz="0.0 0.0 0.0" rpy="${-M_PI/2} 0.0 0.0"/>
-      <geometry>
-        <mesh filename="package://turtlebot_description/meshes/sensors/xtion_pro_stack.dae"/>
-      </geometry>
+      <origin xyz="0.0 0 0.0" rpy="${M_PI*(3/4)} 0.0 ${M_PI/2}"/>
+      <geometry>
+        <mesh filename="package://thorp_bringup/resources/meshes/xtion_mount_a45.stl" scale="0.001 0.001 0.001"/>
+      </geometry>
+      <material name="Black">
+        <color rgba="0.0 0.0 0.0 1.0"/>
+      </material>
     </visual>
     <collision>
       <origin xyz="0.0 0.0 0.0" rpy="0.0 0.0 0.0"/>
       <geometry>
-        <box size="0.028 0.225 0.012"/>
+        <box size="0.02 0.225 0.025"/>
       </geometry>
     </collision>
@@ -130,16 +200,20 @@
     <!-- Ideal extrinsic parameters obtained from robot model -->
     <xacro:if value="$(arg simulation)">
-      <!-- <origin xyz="0.0 -0.025 0.015" rpy="0.0 0.0 0.0"/> -->
-      <origin xyz="0.015 0.01 0.015" rpy="0.0 0.0 0.0"/>
+      <!-- <origin xyz="0.022 0.003 0.002" rpy="0.0 ${M_PI/4} 0.0"/> -->
+      <origin xyz="-0.012 0.003 -0.012" rpy="0.0 0.711982 0.0"/>
     </xacro:if>
     <!-- Extrinsic parameters obtained through arm-camera calibration:
          http://wiki.ros.org/turtlebot_arm_kinect_calibration -->
     <xacro:unless value="$(arg simulation)">
-      <origin xyz="0.015 0.01 0.015" rpy="0.0 0.0 0.0"/>
+      <!-- <origin xyz="-0.0179751 0.0118658 0.022709" rpy="-0.0549698 0.711982 0.00994433"/> -->
+      <!-- <origin xyz="-0.018 0.003 -0.008" rpy="0.0 0.711982 0.0"/> -->
+      <origin xyz="-0.012 0.003 -0.012" rpy="0.0 0.711982 0.0"/>
     </xacro:unless>
   </xtion_camera>
   <!-- Seems like Gazebo kinect plugin needs to use a centered frame instead of separated rgb and depth.
        No idea if this makes any sense, but it works! I also move the optical tf a bit forward to make
-       pointcloud match better the model; this is absolutely arbitrary... -->
+       pointcloud match better the model; this is absolutely arbitrary...
+       TODO: I think I can remove this because I use registered depth images
+        -->
   <xacro:if value="$(arg simulation)">
     <joint name="xtion_gazebo_optical_joint" type="fixed">

File: thorp_bringup/urdf/xtion.urdf.xacro (robot description, xacro)
@@ -28,5 +28,5 @@
     <link name="${name}_link">
       <visual>
-        <origin xyz="-0.015 0.0035 0.004" rpy="0 0 0"/>
+        <origin xyz="0.0 0.0035 0.0375" rpy="0 0 0"/>
         <geometry>
           <mesh filename="package://turtlebot_description/meshes/sensors/xtion_pro_camera.dae"/>

Commit message: Visual origin is parameterized because the "ideal" pose used on simulation and the "working" pose used with the real robot differ
Other minor corrections

File: thorp_bringup/urdf/thorp.urdf.xacro (robot description, xacro)
@@ -103,5 +103,5 @@
   <!-- Mounting plate -->
   <joint name="senz3d_mount_joint" type="fixed">
-    <origin xyz="-0.1124 0.0 ${0.2032 + 0.006 + 0.0515}" rpy="0.0 0.0 0.0"/>
+    <origin xyz="-0.1124 0.0 ${0.006/2 + 0.2032 + 0.0515 + 0.005/2}" rpy="0.0 0.0 0.0"/>
     <parent link="plate_top_link"/>
     <child link="senz3d_mount_link"/>
@@ -149,5 +149,5 @@
   <!-- Seems like Gazebo kinect plugin needs to use a centered frame instead of separated rgb and depth.
        No idea if this makes any sense, but it works! I also move the optical tf a bit forward to make
-       pointcloud match better the model; this is absolutely arbitrary... -->
+       pointcloud match better the model; this is absolutely arbitrary...  TODO sure???  -->
   <xacro:if value="$(arg simulation)">
     <joint name="senz3d_gazebo_optical_joint" type="fixed">
@@ -164,9 +164,9 @@
   <!-- Mounting poles: a pair of top poles -->
   <!-- The Z loc of the upper poles is : 1/2*plate height + 3/2*top pole height -->
-  <stack_top_pole parent="senz3d_mount_link" number="12" x_loc="0.0" y_loc=" 0.098" z_loc="${0.006/2 + 0.2032/2}"/>
-  <stack_top_pole parent="senz3d_mount_link" number="22" x_loc="0.0" y_loc="-0.098" z_loc="${0.006/2 + 0.2032/2}"/>
+  <stack_top_pole parent="senz3d_mount_link" number="12" x_loc="0.0" y_loc=" 0.098" z_loc="${0.005/2 + 0.2032/2}"/>
+  <stack_top_pole parent="senz3d_mount_link" number="22" x_loc="0.0" y_loc="-0.098" z_loc="${0.005/2 + 0.2032/2}"/>
   <!-- Mounting plate -->
   <joint name="xtion_mount_joint" type="fixed">
-    <origin xyz="0.0 0.0 ${0.2032 + 0.006}" rpy="0.0 0.0 0.0"/>
+    <origin xyz="0.0 0.0 ${0.2032 + 0.005/2 + 0.005}" rpy="0.0 0.0 0.0"/>
     <parent link="senz3d_mount_link"/>
     <child link="xtion_mount_link"/>
@@ -200,13 +200,17 @@
     <!-- Ideal extrinsic parameters obtained from robot model -->
     <xacro:if value="$(arg simulation)">
-      <!-- <origin xyz="0.022 0.003 0.002" rpy="0.0 ${M_PI/4} 0.0"/> -->
-      <origin xyz="-0.012 0.003 -0.012" rpy="0.0 0.711982 0.0"/>
+      <origin xyz="0.022 0.003 0.002" rpy="0.0 ${M_PI/4} 0.0"/>
+      <origin xyz="-0.015 0.0035 0.004" rpy="0 0 0"/>    <!-- Visual origin -->
     </xacro:if>
     <!-- Extrinsic parameters obtained through arm-camera calibration:
          http://wiki.ros.org/turtlebot_arm_kinect_calibration -->
     <xacro:unless value="$(arg simulation)">
-      <!-- <origin xyz="-0.0179751 0.0118658 0.022709" rpy="-0.0549698 0.711982 0.00994433"/> -->
-      <!-- <origin xyz="-0.018 0.003 -0.008" rpy="0.0 0.711982 0.0"/> -->
-      <origin xyz="-0.012 0.003 -0.012" rpy="0.0 0.711982 0.0"/>
+      <origin xyz="0.01 0.0 -0.01" rpy="0.0 0.711982 0.02"/>  <!-- p&p try and error  OK for right-side... :o  -->
+      <origin xyz="-0.015 0.007 0.021" rpy="0 0 0"/>    <!-- Visual origin -->
+      <!-- <origin xyz="0.022 0.003 0.002" rpy="0.0 0.711982 0.00994433"/>  ideal from robot model KO -->
+      <!-- <origin xyz="-0.012 -0.006 -0.012" rpy="0.0 0.711982 0.01"/> Fitting pc to robot model  KO -->
+      <!-- <origin xyz="-0.0179751 0.0118658 0.022709" rpy="-0.0549698 0.711982 0.00994433"/>   calib R and T  KO- -->
+      <!-- <origin xyz="0.022 0.0225 0.0" rpy="-0.0292745 0.682572 0.0222799"/>  calib R, measured T  KO-->
+      <!-- <origin xyz="0 0.000831867 0" rpy="-0.0292745 0.682572 0.0222799"/>  calib R, zero T  KO-->
     </xacro:unless>
   </xtion_camera>
@@ -214,6 +218,4 @@
        No idea if this makes any sense, but it works! I also move the optical tf a bit forward to make
        pointcloud match better the model; this is absolutely arbitrary...
-       TODO: I think I can remove this because I use registered depth images
-        -->
   <xacro:if value="$(arg simulation)">
     <joint name="xtion_gazebo_optical_joint" type="fixed">
@@ -223,5 +225,5 @@
     </joint>
     <link name="xtion_gazebo_optical_frame"/>
-  </xacro:if>
+  </xacro:if>        TODO: I think I can remove this because I use registered depth images        -->
   <!-- Sonar sensors forming a half ring centered on (and slightly above) base_link -->
   <joint name="sonars_joint" type="fixed">

File: thorp_bringup/urdf/xtion.urdf.xacro (robot description, xacro)
@@ -5,5 +5,5 @@
   <xacro:property name="asus_xtion_pro_cam_rel_rgb_py" value="-0.0220"/>
   <!-- 3D sensor macro -->
-  <xacro:macro name="xtion_camera" params="parent name *origin">
+  <xacro:macro name="xtion_camera" params="parent name *origin *visual_origin">
     <joint name="${name}_rgb_joint" type="fixed">
       <insert_block name="origin"/>
@@ -26,6 +26,7 @@
     <link name="${name}_link">
       <visual>
-        <origin xyz="-0.015 0.0035 0.004" rpy="0 0 0"/>
-        <!-- <origin xyz="0.0 0.0035 0.0375" rpy="0 0 0"/>    a OJO -->
+        <!-- Visual origin is parameterized because the "ideal" pose used on
+             simulation and the "working" pose used with the real robot differ -->
+        <insert_block name="visual_origin"/>
         <geometry>
           <mesh filename="package://turtlebot_description/meshes/sensors/xtion_pro_camera.dae"/>
