Commit message: Joint limits are not the physical ones; just add a comment on it by now, as I cannot see any problem comming from this!

File: thorp_bringup/urdf/thorp.urdf.xacro (robot description, xacro)
@@ -32,18 +32,17 @@
        TODO: I don't think we need to be that restrictive; do a better problem assessment.
        We also use a deliberately low joints velocity limit to improve safety and precision;
-       The physical limit of the AX-12 is 114 rpm (684 deg/s) -->
+       the physical limit of the AX-12 is 114 rpm (684 deg/s) -->
   <xacro:property name="joints_vlimit" value="0.8"/>
-<!--
-  <xacro:property name="pan_llimit" value="-2.617"/>
-  <xacro:property name="pan_ulimit" value=" 2.617"/>
- -->
+  <!-- <xacro:property name="pan_llimit" value="-2.617"/> -->
+  <!-- <xacro:property name="pan_ulimit" value=" 2.617"/> -->
   <xacro:property name="pan_llimit" value="${-M_PI/2}"/>
   <xacro:property name="pan_ulimit" value="${+M_PI/2}"/>
-  <xacro:property name="shoulder_llimit" value="-2.617"/>
-  <xacro:property name="shoulder_ulimit" value=" 2.617"/>
-  <xacro:property name="elbow_llimit" value=" 0.0"/>
-  <xacro:property name="elbow_ulimit" value=" 2.617"/>
-  <xacro:property name="wrist_llimit" value="-1.745"/>
-  <xacro:property name="wrist_ulimit" value=" 1.745"/>
+  <xacro:property name="shoulder_llimit" value="-2.617"/>  <!-- -150 deg, but physical limit is -2.18 rad (-125 deg) -->
+  <xacro:property name="shoulder_ulimit" value=" 2.617"/>  <!-- +150 deg, but physical limit is +2.18 rad (+125 deg) -->
+  <!-- <xacro:property name="elbow_llimit" value=" -2.617"/> -->
+  <xacro:property name="elbow_llimit" value=" 0.0"/>       <!-- -150 deg, but physical limit is -2.41 rad (-138 deg) -->
+  <xacro:property name="elbow_ulimit" value=" 2.617"/>     <!-- +150 deg, but physical limit is +2.41 rad (+138 deg) -->
+  <xacro:property name="wrist_llimit" value="-1.745"/>     <!-- -100 deg -->
+  <xacro:property name="wrist_ulimit" value=" 1.745"/>     <!-- +100 deg -->
   <turtlebot_arm parent="plate_top_link" color="White" gripper_color="Black"
                  pincher_gripper="false" turtlebot_gripper="true">

Commit message: Calibrate camera (again)

File: thorp_bringup/urdf/thorp.urdf.xacro (robot description, xacro)
@@ -205,6 +205,9 @@
          http://wiki.ros.org/turtlebot_arm_kinect_calibration -->
     <xacro:unless value="$(arg simulation)">
-      <origin xyz="0.01 0.0 -0.01" rpy="0.0 0.711982 0.02"/>  <!-- p&p try and error  OK for right-side... :o  -->
-      <origin xyz="-0.015 0.007 0.021" rpy="0 0 0"/>    <!-- Visual origin -->
+      <!-- Values obtained by calibtrin but compensated after visualization: xyz=-0.01 0.0 -0.003 -->
+      <origin xyz="0.01 -6.25956e-06 0.001" rpy="-0.0319842 0.774615 -0.0120437"/>
+      <!-- Visual origin corrections: undo the rotations for better aesthetics  -->
+      <origin xyz="-0.005 0.006 0.012" rpy="0.0319842 ${M_PI/4 - 0.774615} 0.0120437"/>
+      <!-- <origin xyz="0.01 0.0 -0.01" rpy="0.0 0.711982 0.02"/>  p&p try and error  OK for right-side... :o  -->
       <!-- <origin xyz="0.022 0.003 0.002" rpy="0.0 0.711982 0.00994433"/>  ideal from robot model KO -->
       <!-- <origin xyz="-0.012 -0.006 -0.012" rpy="0.0 0.711982 0.01"/> Fitting pc to robot model  KO -->

Commit message: Add Thorp cannon and a provisional integration on Thorp URDF

File: thorp_bringup/urdf/thorp.urdf.xacro (robot description, xacro)
@@ -16,4 +16,5 @@
   <xacro:include filename="$(find turtlebot_arm_description)/urdf/turtlebot_arm.xacro"/>
   <xacro:include filename="$(find softkinetic_camera)/urdf/senz3d.urdf.xacro"/>
+  <xacro:include filename="$(find thorp_cannon)/urdf/cannon.urdf.xacro"/>
   <xacro:include filename="$(find thorp_bringup)/urdf/thorp_gazebo.urdf.xacro"/>
   <xacro:include filename="$(find thorp_bringup)/urdf/kinect.urdf.xacro"/>
@@ -49,11 +50,19 @@
     <origin xyz="0.10914 0.0295 0.0284"/>
   </turtlebot_arm>
-  <arm_mount parent="arm_base_link" name="arm_mount" color="Black">
+  <arm_mount parent="plate_top_link" name="arm_mount" color="Black">
+    <origin xyz="0.10914 0.0 0.0284" rpy="0.0 0.0 0.0"/>
+  </arm_mount>
+  <arm_mount parent="arm_base_link" name="arm_mount1" color="Black">
     <origin xyz="0.0 0.0 0.0" rpy="0.0 0.0 0.0"/>
   </arm_mount>
+  <arm_mount parent="arm_base_link" name="arm_mount2" color="Black">
+    <origin xyz="0.0 -0.0576 0.0" rpy="0.0 0.0 0.0"/>
+  </arm_mount>
   <stack_bottom_pole parent="arm_base_link" number="10" x_loc=" 0.0"   y_loc=" 0.0288" z_loc="-0.0112"/>
-  <stack_bottom_pole parent="arm_base_link" number="11" x_loc=" 0.0"   y_loc="-0.0288" z_loc="-0.0112"/>
-  <stack_bottom_pole parent="arm_base_link" number="12" x_loc="-0.038" y_loc="-0.0288" z_loc="-0.0112"/>
+  <stack_bottom_pole parent="arm_base_link" number="11" x_loc=" 0.015" y_loc="-0.0288" z_loc="-0.0112"/>
+  <stack_bottom_pole parent="arm_base_link" number="12" x_loc=" 0.0"   y_loc="-0.0864" z_loc="-0.0112"/>
   <stack_bottom_pole parent="arm_base_link" number="13" x_loc="-0.038" y_loc=" 0.0288" z_loc="-0.0112"/>
+  <stack_bottom_pole parent="arm_base_link" number="14" x_loc="-0.038" y_loc="-0.0288" z_loc="-0.0112"/>
+  <stack_bottom_pole parent="arm_base_link" number="15" x_loc="-0.038" y_loc="-0.0864" z_loc="-0.0112"/>
   <!-- Emulate the OpenCM9.04 controller as a box -->
   <joint name="opencm_joint" type="fixed">

Commit message: Integrate the new arm-cannon mount, replacing the small arm mount from turtlebot_arm_description

File: thorp_bringup/urdf/thorp.urdf.xacro (robot description, xacro)
@@ -50,13 +50,32 @@
     <origin xyz="0.10914 0.0295 0.0284"/>
   </turtlebot_arm>
-  <arm_mount parent="plate_top_link" name="arm_mount" color="Black">
-    <origin xyz="0.10914 0.0 0.0284" rpy="0.0 0.0 0.0"/>
-  </arm_mount>
-  <arm_mount parent="arm_base_link" name="arm_mount1" color="Black">
-    <origin xyz="0.0 0.0 0.0" rpy="0.0 0.0 0.0"/>
-  </arm_mount>
-  <arm_mount parent="arm_base_link" name="arm_mount2" color="Black">
-    <origin xyz="0.0 -0.0576 0.0" rpy="0.0 0.0 0.0"/>
-  </arm_mount>
+  <!-- Mount for arm and cannon, set on top of six small poles -->
+  <joint name="arm_mount_joint" type="fixed">
+    <origin xyz="0.10914 0.0 0.042" rpy="0.0 0.0 0.0"/>
+    <parent link="plate_top_link"/>
+    <child link="arm_mount_link"/>
+  </joint>
+  <link name="arm_mount_link">
+    <inertial>
+      <mass value="0.018"/>
+      <origin xyz="0 0 0"/>
+      <inertia ixx="0.000001" ixy="0.0" ixz="0.0"
+               iyy="0.000001" iyz="0.0"
+               izz="0.000001"/>
+    </inertial>
+    <visual>
+      <origin xyz="-0.028 0.0 0.0" rpy="0.0 0.0 -${M_PI/2}"/>
+      <geometry>
+        <mesh filename="package://thorp_bringup/resources/meshes/arm_mount.stl" scale="${M_SCALE} ${M_SCALE} ${M_SCALE}"/>
+      </geometry>
+      <material name="Black"/>
+    </visual>
+    <collision>
+      <origin xyz="-0.01 0.0 0.002" rpy="0.0 0.0 0.0"/>
+      <geometry>
+        <box size="0.074 0.132 0.004"/>
+      </geometry>
+    </collision>
+  </link>
   <stack_bottom_pole parent="arm_base_link" number="10" x_loc=" 0.0"   y_loc=" 0.0288" z_loc="-0.0112"/>
   <stack_bottom_pole parent="arm_base_link" number="11" x_loc=" 0.015" y_loc="-0.0288" z_loc="-0.0112"/>

File: thorp_bringup/urdf/thorp_gazebo.urdf.xacro (robot description, xacro)
@@ -193,4 +193,9 @@
   <Sharp_GP2Y0A21_IR_sim name="r155"/>
   <!-- Gazebo configuration for other structural parts -->
+  <gazebo reference="arm_mount_link">
+    <material>Gazebo/Balck</material>
+    <selfCollide>true</selfCollide>
+    <gravity>true</gravity>
+  </gazebo>
   <gazebo reference="sonars_mount_link">
     <material>Gazebo/Black</material>

File: thorp_cannon/urdf/cannon.urdf.xacro (robot description, xacro)
@@ -6,5 +6,5 @@
   <!-- Emulate the servo as a box and the cannon as a cylinder -->
   <joint name="cannon_servo_joint" type="fixed">
-    <origin xyz="-0.008 -0.003 -0.0042" rpy="0.0 0.0 0.0"/>
+    <origin xyz="-0.008 -0.003 -0.0195" rpy="0.0 0.0 0.0"/>
     <parent link="arm_mount_link"/>
     <child link="cannon_servo_link"/>

Commit message: Slight changes to arm mount after first 3D print

File: thorp_bringup/urdf/thorp.urdf.xacro (robot description, xacro)
@@ -79,5 +79,5 @@
   </link>
   <stack_bottom_pole parent="arm_base_link" number="10" x_loc=" 0.0"   y_loc=" 0.0288" z_loc="-0.0112"/>
-  <stack_bottom_pole parent="arm_base_link" number="11" x_loc=" 0.015" y_loc="-0.0288" z_loc="-0.0112"/>
+  <stack_bottom_pole parent="arm_base_link" number="11" x_loc=" 0.014" y_loc="-0.0288" z_loc="-0.0112"/>
   <stack_bottom_pole parent="arm_base_link" number="12" x_loc=" 0.0"   y_loc="-0.0864" z_loc="-0.0112"/>
   <stack_bottom_pole parent="arm_base_link" number="13" x_loc="-0.038" y_loc=" 0.0288" z_loc="-0.0112"/>

File: thorp_cannon/urdf/cannon.urdf.xacro (robot description, xacro)
@@ -6,5 +6,5 @@
   <!-- Emulate the servo as a box and the cannon as a cylinder -->
   <joint name="cannon_servo_joint" type="fixed">
-    <origin xyz="-0.008 -0.003 -0.0195" rpy="0.0 0.0 0.0"/>
+    <origin xyz="-0.009 -0.002 -0.0195" rpy="0.0 0.0 0.0"/>
     <parent link="arm_mount_link"/>
     <child link="cannon_servo_link"/>
