Commit message: Remove useless tag

File: thorp_description/urdf/cannon.urdf.xacro (robot description, xacro)
@@ -63,5 +63,4 @@
     <limit effort="30" velocity="0.10471975512" lower="-0.523598775598" upper="0.523598775598"/>
     <!-- 6 degrees/s, +/-30 degrees operational range -->
-    <dynamics friction="0.13"/>  <!-- no idea -->
     <origin xyz="0.0 -0.015 0.0" rpy="0.0 0.0 0.0"/>
     <parent link="cannon_shaft_link"/>

Commit message: Increase cannon tilt speed, closer to the hw

File: thorp_description/urdf/cannon.urdf.xacro (robot description, xacro)
@@ -61,6 +61,7 @@
   <joint name="cannon_joint" type="revolute">
     <axis xyz="0 -1 0"/>
-    <limit effort="30" velocity="0.10471975512" lower="-0.523598775598" upper="0.523598775598"/>
-    <!-- 6 degrees/s, +/-30 degrees operational range -->
+    <limit effort="1.0" velocity="5.0" lower="${-M_PI/10}" upper="${+M_PI/10}"/>
+    <!-- 300 degrees/s (specs say 600/s, but then I cannot see the cannon rotate in gazebo),
+         limits: +/-18 degrees operational range (servo limits are +/-30 degrees, I think) -->
     <origin xyz="0.0 -0.015 0.0" rpy="0.0 0.0 0.0"/>
     <parent link="cannon_shaft_link"/>

Commit message: Make inertias more realistic and simpler with box_inertia macro

File: thorp_description/urdf/cannon.urdf.xacro (robot description, xacro)
@@ -18,19 +18,12 @@
       <material name="Black"/>
     </visual>
-    <collision>
-      <origin xyz="0.0 0.006 0.0" rpy="0.0 0.0 0.0"/>
-      <geometry>
-        <box size="0.022 0.022 0.012"/>
-      </geometry>
-    </collision>
-    <inertial>
-      <mass value="0.01"/>
-      <origin xyz="0 0 0"/>
-      <inertia ixx="0.0001" ixy="0.0" ixz="0.0"
-               iyy="0.0001" iyz="0.0"
-               izz="0.0001"/>
-    </inertial>
+    <xacro:box_inertia length="0.022" width="0.022" height="0.012" mass="0.01"/>
+    <!-- covered under the arm mount, so no need for collision -->
   </link>
-  <joint name="cannon_shaft_joint" type="fixed">
+  <joint name="cannon_joint" type="revolute">
+    <axis xyz="0 -1 0"/>
+    <limit effort="1.0" velocity="5.0" lower="${-M_PI/10}" upper="${+M_PI/10}"/>
+    <!-- 300 degrees/s (specs say 600/s, but then I cannot see the cannon rotate in gazebo),
+         limits: +/-18 degrees operational range (servo limits are +/-30 degrees, I think) -->
     <origin xyz="0.006 -0.015 0.0" rpy="0.0 0.0 0.0"/>
     <parent link="cannon_servo_link"/>
@@ -45,23 +38,7 @@
       <material name="Black"/>
     </visual>
-    <collision>
-      <origin xyz="0.0 0.002 0.0" rpy="${+M_PI/2} 0.0 0.0"/>
-      <geometry>
-        <cylinder radius="0.002" length="0.016"/>
-      </geometry>
-    </collision>
-    <inertial>
-      <mass value="0.002"/>
-      <origin xyz="0 0 0"/>
-      <inertia ixx="0.0001" ixy="0.0" ixz="0.0"
-               iyy="0.0001" iyz="0.0"
-               izz="0.0001"/>
-    </inertial>
+    <!-- very small and light, so we don't need collision and inertial -->
   </link>
-  <joint name="cannon_joint" type="revolute">
-    <axis xyz="0 -1 0"/>
-    <limit effort="1.0" velocity="5.0" lower="${-M_PI/10}" upper="${+M_PI/10}"/>
-    <!-- 300 degrees/s (specs say 600/s, but then I cannot see the cannon rotate in gazebo),
-         limits: +/-18 degrees operational range (servo limits are +/-30 degrees, I think) -->
+  <joint name="cannon_shaft_joint" type="fixed">
     <origin xyz="0.0 -0.015 0.0" rpy="0.0 0.0 0.0"/>
     <parent link="cannon_shaft_link"/>
@@ -82,11 +59,6 @@
       </geometry>
     </collision>
-    <inertial>
-      <mass value="0.01"/>
-      <origin xyz="0.01 0.0 0.0"/>
-      <inertia ixx="0.0001" ixy="0.0" ixz="0.0"
-               iyy="0.0001" iyz="0.0"
-               izz="0.0001"/>
-    </inertial>
+    <xacro:box_inertia length="0.03" width="0.02" height="0.02" mass="0.01" x="0.01"/>
+    <!-- should be a cylinder... but is very light to bother -->
   </link>
   <!-- Emulate the six cannon tubes with two cylinders, the second a bit smaller and transparent -->

File: thorp_description/urdf/thorp.urdf.xacro (robot description, xacro)
@@ -61,11 +61,4 @@
   </joint>
   <link name="arm_mount_link">
-    <inertial>
-      <mass value="0.048"/>
-      <origin xyz="0 0 0"/>
-      <inertia ixx="0.000001" ixy="0.0" ixz="0.0"
-               iyy="0.000001" iyz="0.0"
-               izz="0.000001"/>
-    </inertial>
     <visual>
       <origin xyz="-0.028 0.0 0.0" rpy="0.0 0.0 -${M_PI/2}"/>
@@ -81,4 +74,5 @@
       </geometry>
     </collision>
+    <xacro:box_inertia length="0.074" width="0.132" height="0.004" mass="0.048"/>
   </link>
   <xacro:stack_bottom_pole parent="arm_base_link" number="10" x_loc=" 0.0"   y_loc=" 0.0288" z_loc="-0.0112"/>
@@ -88,5 +82,5 @@
   <xacro:stack_bottom_pole parent="arm_base_link" number="14" x_loc="-0.038" y_loc="-0.0288" z_loc="-0.0112"/>
   <xacro:stack_bottom_pole parent="arm_base_link" number="15" x_loc="-0.038" y_loc="-0.0864" z_loc="-0.0112"/>
-  <!-- Emulate the OpenCM9.04 controller as a box -->
+  <!-- Emulate the OpenCM9.04 controller as a box  TODO: replaced with ... -->
   <joint name="opencm_joint" type="fixed">
     <origin xyz="0.045 0.03 0.008" rpy="0.0 0.0 0.0"/>
@@ -110,11 +104,5 @@
       </geometry>
     </collision>
-    <inertial>
-      <mass value="0.01"/>
-      <origin xyz="0 0 0"/>
-      <inertia ixx="0.0001" ixy="0.0" ixz="0.0"
-               iyy="0.0001" iyz="0.0"
-               izz="0.0001"/>
-    </inertial>
+    <xacro:box_inertia length="0.027" width="0.0665" height="0.01" mass="0.013"/>
   </link>
   <!-- Arm IR sensor link, mounted below the arm mount and pointing forward -->
@@ -151,11 +139,5 @@
       </geometry>
     </collision>
-    <inertial>
-      <mass value="0.040"/>
-      <origin xyz="0 0 0"/>
-      <inertia ixx="0.0001" ixy="0.0" ixz="0.0"
-               iyy="0.0001" iyz="0.0"
-               izz="0.0001"/>
-    </inertial>
+    <xacro:box_inertia length="0.03" width="0.22" height="0.006" mass="0.040"/>
   </link>
   <!-- The camera itself -->
@@ -197,6 +179,6 @@
   <xacro:stack_middle_pole parent="senz3d_mount_link" number="11" x_loc="0.0" y_loc=" 0.098" z_loc="${0.005/2 + 0.2032 + 0.0608/2}"/>
   <xacro:stack_middle_pole parent="senz3d_mount_link" number="21" x_loc="0.0" y_loc="-0.098" z_loc="${0.005/2 + 0.2032 + 0.0608/2}"/>
-  <!-- Mounting plate. The Z loc of the upper middle poles is : -->
-  <!--   1/2*Senz3D mounting plate height + middle pole height (without screw) + top pole height + mounting's poles housing -->
+  <!-- Mounting plate. The Z loc of the upper middle poles is: -->
+  <!--   1/2 * Senz3D mounting plate height + middle pole height (without screw) + top pole height + mounting's poles housing -->
   <joint name="xtion_mount_joint" type="fixed">
     <origin xyz="0.0 0.0 ${0.005/2 + 0.05 + 0.2032 + 0.005}" rpy="0.0 0.0 0.0"/>
@@ -220,11 +202,5 @@
       </geometry>
     </collision>
-    <inertial>
-      <mass value="0.040"/>
-      <origin xyz="0 0 0"/>
-        <inertia ixx="0.0001" ixy="0.0" ixz="0.0"
-                 iyy="0.0001" iyz="0.0"
-                 izz="0.0001"/>
-    </inertial>
+    <xacro:box_inertia length="0.02" width="0.225" height="0.025" mass="0.040"/>
   </link>
   <!-- The camera itself -->
@@ -260,11 +236,4 @@
   </joint>
   <link name="sonars_mount_link">
-    <inertial>
-      <mass value="0.22"/>
-      <origin xyz="0 0 0"/>
-      <inertia ixx="0.0001" ixy="0.0" ixz="0.0"
-               iyy="0.0001" iyz="0.0"
-               izz="0.0001"/>
-    </inertial>
     <visual>
       <origin xyz="0.0 0.0 -0.0586" rpy="${-M_PI/2} -${M_PI} ${-M_PI/2}"/>
@@ -273,10 +242,14 @@
       </geometry>
     </visual>
-    <collision>
-      <origin xyz="-0.01 0.0 0.0165" rpy="0.0 0.0 0.0"/>
-      <geometry>
-        <box size="0.074 0.074 0.004"/>
-      </geometry>
-    </collision>
+    <xacro:box_inertia length="0.17" width="0.325" height="0.035" mass="0.3" x="0.068"/>
+    <!-- Include also the 11 EZ2 and the arduino board: 0.22 + 11 * 0.005 + 0.025 = 0.3 -->
+    <!-- We don't need collision, as this part is mostly covered by kobuki base cylinder
+    <collision>
+      <origin xyz="0.068 0.0 0.0" rpy="0.0 0.0 0.0"/>
+      <geometry>
+        <box size="0.17 0.325 0.035"/>
+      </geometry>
+    </collision>
+-->
   </link>
   <xacro:macro name="LV_MaxSonar_EZ2_sensor" params="name parent x_loc y_loc yaw">
@@ -287,11 +260,5 @@
     </joint>
     <link name="s_${name}_link">
-      <inertial>
-        <mass value="0.001"/>
-        <origin xyz="0 0 0" rpy="0 0 0"/>
-        <inertia ixx="0.000001" ixy="0.0" ixz="0.0"
-                 iyy="0.000001" iyz="0.0"
-                 izz="0.000001"/>
-      </inertial>
+    <!-- Collision and inertial already added to the mount -->
       <visual>
         <origin xyz="0 0 0" rpy="0 0 0" />
@@ -300,13 +267,7 @@
         </geometry>
       </visual>
-      <collision>
-        <origin xyz="0 0 0" rpy="0 0 0"/>
-        <geometry>
-          <box size="0.01 0.01 0.01"/>
-        </geometry>
-      </collision>
     </link>
   </xacro:macro>
-  <xacro:LV_MaxSonar_EZ2_sensor name="m90" parent="sonars_mount_link" x_loc="0.0"    y_loc="-0.1380" yaw="-1.57080"/>
+  <xacro:LV_MaxSonar_EZ2_sensor  name="m90" parent="sonars_mount_link" x_loc="0.0"    y_loc="-0.1380" yaw="-1.57080"/>
   <xacro:LV_MaxSonar_EZ2_sensor name="m72" parent="sonars_mount_link" x_loc="0.0426" y_loc="-0.1312" yaw="-1.25664"/>
   <xacro:LV_MaxSonar_EZ2_sensor name="m54" parent="sonars_mount_link" x_loc="0.0811" y_loc="-0.1116" yaw="-0.94248"/>

Commit message: Restore cannon_joint as the actuated one, so gazebo cannon uses cannon_link

File: thorp_description/urdf/cannon.urdf.xacro (robot description, xacro)
@@ -21,9 +21,5 @@
     <!-- covered under the arm mount, so no need for collision -->
   </link>
-  <joint name="cannon_joint" type="revolute">
-    <axis xyz="0 -1 0"/>
-    <limit effort="1.0" velocity="5.0" lower="${-M_PI/10}" upper="${+M_PI/10}"/>
-    <!-- 300 degrees/s (specs say 600/s, but then I cannot see the cannon rotate in gazebo),
-         limits: +/-18 degrees operational range (servo limits are +/-30 degrees, I think) -->
+  <joint name="cannon_shaft_joint" type="fixed">
     <origin xyz="0.006 -0.015 0.0" rpy="0.0 0.0 0.0"/>
     <parent link="cannon_servo_link"/>
@@ -38,7 +34,12 @@
       <material name="Black"/>
     </visual>
-    <!-- very small and light, so we don't need collision and inertial -->
+    <xacro:cylinder_inertia radius="0.002" height="0.016" mass="0.001"/>
+    <!-- covered under the arm mount, so no need for collision -->
   </link>
-  <joint name="cannon_shaft_joint" type="fixed">
+  <joint name="cannon_joint" type="revolute">
+    <axis xyz="0 -1 0"/>
+    <limit effort="1.0" velocity="5.0" lower="${-M_PI/10}" upper="${+M_PI/10}"/>
+    <!-- 300 degrees/s (specs say 600/s, but then I cannot see the cannon rotate in gazebo),
+         limits: +/-18 degrees operational range (servo limits are +/-30 degrees, I think) -->
     <origin xyz="0.0 -0.015 0.0" rpy="0.0 0.0 0.0"/>
     <parent link="cannon_shaft_link"/>
@@ -59,6 +60,5 @@
       </geometry>
     </collision>
-    <xacro:box_inertia length="0.03" width="0.02" height="0.02" mass="0.01" x="0.01"/>
-    <!-- should be a cylinder... but is very light to bother -->
+    <xacro:cylinder_inertia radius="0.01" height="0.03" mass="0.01" x="0.01" P="${+M_PI/2}"/>
   </link>
   <!-- Emulate the six cannon tubes with two cylinders, the second a bit smaller and transparent -->

Commit message: Reduce cannon collision model so it doesn't hit the table

File: thorp_description/urdf/cannon.urdf.xacro (robot description, xacro)
@@ -55,7 +55,7 @@
     </visual>
     <collision>
-      <origin xyz="0.019 0.0 0.0" rpy="0.0 ${+M_PI/2} 0.0"/>
+      <origin xyz="0.022 0.0 0.0" rpy="0.0 ${+M_PI/2} 0.0"/>
       <geometry>
-        <cylinder radius="0.01" length="0.066"/>
+        <cylinder radius="0.007" length="0.054"/>
       </geometry>
     </collision>
