Commit message: Port thorp_description to ROS 2
The generated URDF is identical to the Noetic one (every link, joint,
origin, limit, visual, collision, inertial and material), both with and
without simulation:=true; only the Gazebo Classic <gazebo> and
<transmission> elements are gone, to be replaced when porting the
simulation.

- Copy the TurtleBot 2 (Kobuki base, hexagon stacks, Kinect), TurtleBot
  arm and sonar description files Thorp used on Noetic, as none of those
  packages has a Jazzy release; README records sources and changes
- Move the ir_cannon_link frame from thorp_gazebo.urdf.xacro, which is
  no longer included, to cannon.urdf.xacro
- Set the arm's M_PI to full precision, so the result doesn't depend on
  the include order
- Replace the dangling orig_arm_mount.stl symlink with the copied mesh
- Add display.launch.py and an RViz config to view the model

Co-Authored-By: Claude Opus 5.5 <noreply@anthropic.com>
Claude-Session: https://claude.ai/code/session_01Sj6Jp6D5WDzTQ3UthEdter

File: thorp_description/urdf/cannon.urdf.xacro (robot description, xacro)
@@ -101,3 +101,10 @@
   <xacro:cannon_tube parent="cannon_link" number="5" y_loc="-0.002200" z_loc="-0.003811"/>
   <xacro:cannon_tube parent="cannon_link" number="6" y_loc=" 0.002200" z_loc="-0.003811"/>
+  <!-- Frame for a fake range sensor used to see where the cannon is pointing to -->
+  <joint name="ir_cannon_joint" type="fixed">
+    <origin xyz="0.035 0.0 0.0"/>
+    <parent link="cannon_link"/>
+    <child link="ir_cannon_link"/>
+  </joint>
+  <link name="ir_cannon_link"/>
 </robot>

File: thorp_description/urdf/kinect.urdf.xacro (robot description, xacro)
@@ -1,5 +1,5 @@
 <?xml version="1.0"?>
 <robot name="kinect_camera" xmlns:xacro="http://ros.org/wiki/xacro">
-  <xacro:include filename="$(find turtlebot_description)/urdf/turtlebot_properties.urdf.xacro"/>
+  <xacro:include filename="$(find thorp_description)/urdf/turtlebot/turtlebot_properties.urdf.xacro"/>
   <xacro:property name="kinect_cam_py" value="-0.0125"/>
   <!-- 3D sensor macro -->
@@ -29,5 +29,5 @@
        <origin xyz="-0.031 ${-kinect_cam_py} -0.016" rpy="0 0 ${M_PI/2}"/>
         <geometry>
-         <mesh filename="package://turtlebot_description/meshes/sensors/kinect.dae"/>
+         <mesh filename="package://thorp_description/meshes/turtlebot/sensors/kinect.dae"/>
         </geometry>
       </visual>
@@ -61,6 +61,4 @@
     </joint>
     <link name="${name}_depth_optical_frame"/>
-    <!-- RGBD sensor for simulation -->
-    <xacro:thorp_sim_3dsensor name="${name}" depth_registration="true"/>
   </xacro:macro>
 </robot>

File: thorp_description/urdf/standalone_arm.urdf.xacro (robot description, xacro)
@@ -5,5 +5,5 @@
     xmlns:interface="http://playerstage.sourceforge.net/gazebo/xmlschema/#interface">
     <!-- Included URDF Files -->
-    <xacro:include filename="$(find turtlebot_arm_description)/urdf/turtlebot_arm.xacro" />
+    <xacro:include filename="$(find thorp_description)/urdf/turtlebot_arm/turtlebot_arm.xacro" />
       <!-- Used for fixing robot to Gazebo 'base_link' -->
   <link name="world"/>

File: thorp_description/urdf/thorp.urdf.xacro (robot description, xacro)
@@ -14,9 +14,7 @@
 -->
 <robot name="Thorp" xmlns:xacro="http://ros.org/wiki/xacro">
-  <xacro:include filename="$(find turtlebot_description)/urdf/turtlebot_common_library.urdf.xacro"/>
-  <xacro:include filename="$(find turtlebot_description)/urdf/stacks/hexagons.urdf.xacro"/>
-  <xacro:include filename="$(find turtlebot_arm_description)/urdf/turtlebot_arm.xacro"/>
-  <xacro:include filename="$(find kobuki_description)/urdf/kobuki.urdf.xacro"/>
-  <xacro:include filename="$(find thorp_description)/urdf/thorp_gazebo.urdf.xacro"/>
+  <xacro:include filename="$(find thorp_description)/urdf/turtlebot/kobuki.urdf.xacro"/>
+  <xacro:include filename="$(find thorp_description)/urdf/turtlebot/hexagons.urdf.xacro"/>
+  <xacro:include filename="$(find thorp_description)/urdf/turtlebot_arm/turtlebot_arm.xacro"/>
   <xacro:include filename="$(find thorp_description)/urdf/cannon.urdf.xacro"/>
   <xacro:include filename="$(find thorp_description)/urdf/kinect.urdf.xacro"/>
@@ -258,5 +256,5 @@
         <origin xyz="0 0 0" rpy="0 0 0" />
         <geometry>
-          <mesh filename="package://hector_sensors_description/meshes/sonar_sensor/max_sonar_ez4.dae" scale="1.1 1.1 1.1"/>/>
+          <mesh filename="package://thorp_description/meshes/sensors/max_sonar_ez4.dae" scale="1.1 1.1 1.1"/>
         </geometry>
       </visual>

File: thorp_description/urdf/xtion.urdf.xacro (robot description, xacro)
@@ -59,6 +59,4 @@
     </joint>
     <link name="${name}_depth_optical_frame"/>
-    <!-- RGBD sensor for simulation -->
-    <xacro:thorp_sim_3dsensor name="${name}" depth_registration="true"/>
   </xacro:macro>
 </robot>
