Commit message: Adapt to new xacro files Processing Order using flag --inorder. I also moved cannon xacro file to the new thorp_description package

File: thorp_description/urdf/thorp.urdf.xacro (robot description, xacro)
@@ -9,4 +9,5 @@
     - 5 IR sensors
     - Turtlebot arm
+    - Rocket launcher
     - Auxiliary 3D sensor (Creative Senz3D)
     - Manipulation 3D sensor (Asus Xtion Pro)
@@ -16,6 +17,6 @@
   <xacro:include filename="$(find turtlebot_arm_description)/urdf/turtlebot_arm.xacro"/>
   <xacro:include filename="$(find softkinetic_camera)/urdf/senz3d.urdf.xacro"/>
-  <xacro:include filename="$(find thorp_cannon)/urdf/cannon.urdf.xacro"/>
   <xacro:include filename="$(find thorp_description)/urdf/thorp_gazebo.urdf.xacro"/>
+  <xacro:include filename="$(find thorp_description)/urdf/cannon.urdf.xacro"/>
   <xacro:include filename="$(find thorp_description)/urdf/kinect.urdf.xacro"/>
   <xacro:include filename="$(find thorp_description)/urdf/xtion.urdf.xacro"/>
@@ -283,15 +284,4 @@
     </collision>
   </link>
-  <LV_MaxSonar_EZ2_sensor name="m90" parent="sonars_mount_link" x_loc="0.0"    y_loc="-0.1380" yaw="-1.57080"/>
-  <LV_MaxSonar_EZ2_sensor name="m72" parent="sonars_mount_link" x_loc="0.0426" y_loc="-0.1312" yaw="-1.25664"/>
-  <LV_MaxSonar_EZ2_sensor name="m54" parent="sonars_mount_link" x_loc="0.0811" y_loc="-0.1116" yaw="-0.94248"/>
-  <LV_MaxSonar_EZ2_sensor name="m36" parent="sonars_mount_link" x_loc="0.1116" y_loc="-0.0811" yaw="-0.62832"/>
-  <LV_MaxSonar_EZ2_sensor name="m18" parent="sonars_mount_link" x_loc="0.1312" y_loc="-0.0426" yaw="-0.31416"/>
-  <LV_MaxSonar_EZ2_sensor name="0"   parent="sonars_mount_link" x_loc="0.138"  y_loc=" 0.0"    yaw=" 0.0"/>
-  <LV_MaxSonar_EZ2_sensor name="p18" parent="sonars_mount_link" x_loc="0.1312" y_loc="+0.0426" yaw="+0.31416"/>
-  <LV_MaxSonar_EZ2_sensor name="p36" parent="sonars_mount_link" x_loc="0.1116" y_loc="+0.0811" yaw="+0.62832"/>
-  <LV_MaxSonar_EZ2_sensor name="p54" parent="sonars_mount_link" x_loc="0.0811" y_loc="+0.1116" yaw="+0.94248"/>
-  <LV_MaxSonar_EZ2_sensor name="p72" parent="sonars_mount_link" x_loc="0.0426" y_loc="+0.1312" yaw="+1.25664"/>
-  <LV_MaxSonar_EZ2_sensor name="p90" parent="sonars_mount_link" x_loc="0.0"    y_loc="+0.1380" yaw="+1.57080"/>
   <xacro:macro name="LV_MaxSonar_EZ2_sensor" params="name parent x_loc y_loc yaw">
     <joint name="s_${name}_joint" type="fixed">
@@ -322,4 +312,15 @@
     </link>
   </xacro:macro>
+  <LV_MaxSonar_EZ2_sensor name="m90" parent="sonars_mount_link" x_loc="0.0"    y_loc="-0.1380" yaw="-1.57080"/>
+  <LV_MaxSonar_EZ2_sensor name="m72" parent="sonars_mount_link" x_loc="0.0426" y_loc="-0.1312" yaw="-1.25664"/>
+  <LV_MaxSonar_EZ2_sensor name="m54" parent="sonars_mount_link" x_loc="0.0811" y_loc="-0.1116" yaw="-0.94248"/>
+  <LV_MaxSonar_EZ2_sensor name="m36" parent="sonars_mount_link" x_loc="0.1116" y_loc="-0.0811" yaw="-0.62832"/>
+  <LV_MaxSonar_EZ2_sensor name="m18" parent="sonars_mount_link" x_loc="0.1312" y_loc="-0.0426" yaw="-0.31416"/>
+  <LV_MaxSonar_EZ2_sensor name="0"   parent="sonars_mount_link" x_loc="0.138"  y_loc=" 0.0"    yaw=" 0.0"/>
+  <LV_MaxSonar_EZ2_sensor name="p18" parent="sonars_mount_link" x_loc="0.1312" y_loc="+0.0426" yaw="+0.31416"/>
+  <LV_MaxSonar_EZ2_sensor name="p36" parent="sonars_mount_link" x_loc="0.1116" y_loc="+0.0811" yaw="+0.62832"/>
+  <LV_MaxSonar_EZ2_sensor name="p54" parent="sonars_mount_link" x_loc="0.0811" y_loc="+0.1116" yaw="+0.94248"/>
+  <LV_MaxSonar_EZ2_sensor name="p72" parent="sonars_mount_link" x_loc="0.0426" y_loc="+0.1312" yaw="+1.25664"/>
+  <LV_MaxSonar_EZ2_sensor name="p90" parent="sonars_mount_link" x_loc="0.0"    y_loc="+0.1380" yaw="+1.57080"/>
   <!-- IR sensor links, pointing at -155, pi, pi and 155 degrees -->
   <joint name="ir_l155_joint" type="fixed">

File: thorp_description/urdf/thorp_gazebo.urdf.xacro (robot description, xacro)
@@ -194,5 +194,5 @@
   <!-- Gazebo configuration for other structural parts -->
   <gazebo reference="arm_mount_link">
-    <material>Gazebo/Balck</material>
+    <material>Gazebo/Black</material>
     <selfCollide>true</selfCollide>
     <gravity>true</gravity>
@@ -214,4 +214,9 @@
   </gazebo>
   <gazebo reference="opencm_link">
+    <material>Gazebo/Black</material>
+    <selfCollide>true</selfCollide>
+    <gravity>true</gravity>
+  </gazebo>
+  <gazebo reference="cannon_link">
     <material>Gazebo/Black</material>
     <selfCollide>true</selfCollide>

File: thorp_description/urdf/xtion.urdf.xacro (robot description, xacro)
@@ -7,5 +7,5 @@
   <xacro:macro name="xtion_camera" params="parent name *origin *visual_origin">
     <joint name="${name}_rgb_joint" type="fixed">
-      <insert_block name="origin"/>
+      <xacro:insert_block name="origin"/>
       <parent link="${parent}"/>
       <child link="${name}_rgb_frame"/>
@@ -28,5 +28,5 @@
         <!-- Visual origin is parameterized because the "ideal" pose used on
              simulation and the "working" pose used with the real robot differ -->
-        <insert_block name="visual_origin"/>
+        <xacro:insert_block name="visual_origin"/>
         <geometry>
           <mesh filename="package://turtlebot_description/meshes/sensors/xtion_pro_camera.dae"/>

Commit message: Fix link weight

File: thorp_description/urdf/thorp.urdf.xacro (robot description, xacro)
@@ -62,5 +62,5 @@
   <link name="arm_mount_link">
     <inertial>
-      <mass value="0.018"/>
+      <mass value="0.048"/>
       <origin xyz="0 0 0"/>
       <inertia ixx="0.000001" ixy="0.0" ixz="0.0"

Commit message: Add a more solid Xtion mount

File: thorp_description/urdf/thorp.urdf.xacro (robot description, xacro)
@@ -205,7 +205,7 @@
   <link name="xtion_mount_link">
     <visual>
-      <origin xyz="0.0 0 0.0" rpy="${M_PI*(3/4)} 0.0 ${M_PI/2}"/>
-      <geometry>
-        <mesh filename="package://thorp_description/meshes/xtion_mount_a45.stl" scale="0.001 0.001 0.001"/>
+      <origin xyz="0.0 0 0.0" rpy="0.0 0.0 ${M_PI/2}"/>
+      <geometry>
+        <mesh filename="package://thorp_description/meshes/xtion_mount.stl" scale="0.001 0.001 0.001"/>
       </geometry>
       <material name="Black">

Commit message: Use fitting pc to robot model instead of calibrated extrinsics for Xtion pose

File: thorp_description/urdf/thorp.urdf.xacro (robot description, xacro)
@@ -126,13 +126,10 @@
   <link name="ir_arm_link"/>
   <!-- Auxiliary Senz3D camera plus mounting on Thorp -->
-  <!-- Mounting poles: two columns made with one top and one middle poles stacked -->
-  <!-- The Z loc of the upper poles is : 1/2*plate height + top pole height + 1/2*middle pole height (without screw) -->
+  <!-- Mounting poles: a pair of top poles -->
   <stack_top_pole parent="plate_top_link" number="10" x_loc="-0.1124" y_loc=" 0.098" z_loc="${0.006/2 + 0.2032/2}"/>
   <stack_top_pole parent="plate_top_link" number="20" x_loc="-0.1124" y_loc="-0.098" z_loc="${0.006/2 + 0.2032/2}"/>
-  <stack_middle_pole parent="plate_top_link" number="11" x_loc="-0.1124" y_loc=" 0.098" z_loc="${0.006/2 + 0.2032 + 0.0608/2}"/>
-  <stack_middle_pole parent="plate_top_link" number="21" x_loc="-0.1124" y_loc="-0.098" z_loc="${0.006/2 + 0.2032 + 0.0608/2}"/>
   <!-- Mounting plate -->
   <joint name="senz3d_mount_joint" type="fixed">
-    <origin xyz="-0.1124 0.0 ${0.006/2 + 0.2032 + 0.0515 + 0.005/2}" rpy="0.0 0.0 0.0"/>
+    <origin xyz="-0.1124 0.0 ${0.006/2 + 0.2032 + 0.005/2}" rpy="0.0 0.0 0.0"/>
     <parent link="plate_top_link"/>
     <child link="senz3d_mount_link"/>
@@ -192,12 +189,16 @@
     <origin xyz="0.0 0.0 0.0" rpy="0.0 0.0 0.0"/>
   </sensor_senz3d>
-  <!-- Manipulation Asus Xtion Pro camera mounted on top of the Senz3D's mounting plate-->
-  <!-- Mounting poles: a pair of top poles -->
-  <!-- The Z loc of the upper poles is : 1/2*plate height + 3/2*top pole height -->
+  <!-- Manipulation Asus Xtion Pro camera mounted on top of the Senz3D's mounting plate -->
+  <!-- Mounting poles: two columns made with one top and one middle poles stacked -->
+  <!-- The Z loc of the lower top poles is : 1/2*plate height + 3/2*top pole height -->
+  <!-- The Z loc of the upper middle poles is : 1/2*plate height + top pole height + 1/2*middle pole height (with screw) -->
   <stack_top_pole parent="senz3d_mount_link" number="12" x_loc="0.0" y_loc=" 0.098" z_loc="${0.005/2 + 0.2032/2}"/>
   <stack_top_pole parent="senz3d_mount_link" number="22" x_loc="0.0" y_loc="-0.098" z_loc="${0.005/2 + 0.2032/2}"/>
-  <!-- Mounting plate -->
+  <stack_middle_pole parent="senz3d_mount_link" number="11" x_loc="0.0" y_loc=" 0.098" z_loc="${0.005/2 + 0.2032 + 0.0608/2}"/>
+  <stack_middle_pole parent="senz3d_mount_link" number="21" x_loc="0.0" y_loc="-0.098" z_loc="${0.005/2 + 0.2032 + 0.0608/2}"/>
+  <!-- Mounting plate. The Z loc of the upper middle poles is : -->
+  <!--   1/2*Senz3D mounting plate height + middle pole height (without screw) + top pole height + mounting's poles housing -->
   <joint name="xtion_mount_joint" type="fixed">
-    <origin xyz="0.0 0.0 ${0.2032 + 0.005/2 + 0.005}" rpy="0.0 0.0 0.0"/>
+    <origin xyz="0.0 0.0 ${0.005/2 + 0.05 + 0.2032 + 0.005}" rpy="0.0 0.0 0.0"/>
     <parent link="senz3d_mount_link"/>
     <child link="xtion_mount_link"/>
@@ -231,20 +232,12 @@
     <!-- Ideal extrinsic parameters obtained from robot model -->
     <xacro:if value="$(arg simulation)">
-      <origin xyz="0.022 0.003 0.002" rpy="0.0 ${M_PI/4} 0.0"/>
+      <origin xyz="0.022 0.003 0.002" rpy="0.0 0.694626 0.0"/>
       <origin xyz="-0.015 0.0035 0.004" rpy="0 0 0"/>    <!-- Visual origin -->
     </xacro:if>
-    <!-- Extrinsic parameters obtained through arm-camera calibration:
-         http://wiki.ros.org/turtlebot_arm_kinect_calibration -->
+    <!-- Extrinsic parameters obtained by fitting the visible pc to robot model -->
     <xacro:unless value="$(arg simulation)">
-      <!-- Values obtained by calibtrin but compensated after visualization: xyz=-0.01 0.0 -0.003 -->
-      <origin xyz="0.01 -6.25956e-06 0.001" rpy="-0.0319842 0.774615 -0.0120437"/>
+      <origin xyz="-0.012 0.0065 -0.012" rpy="0.0 0.697357 0.0"/>
       <!-- Visual origin corrections: undo the rotations for better aesthetics  -->
-      <origin xyz="-0.005 0.006 0.012" rpy="0.0319842 ${M_PI/4 - 0.774615} 0.0120437"/>
-      <!-- <origin xyz="0.01 0.0 -0.01" rpy="0.0 0.711982 0.02"/>  p&p try and error  OK for right-side... :o  -->
-      <!-- <origin xyz="0.022 0.003 0.002" rpy="0.0 0.711982 0.00994433"/>  ideal from robot model KO -->
-      <!-- <origin xyz="-0.012 -0.006 -0.012" rpy="0.0 0.711982 0.01"/> Fitting pc to robot model  KO -->
-      <!-- <origin xyz="-0.0179751 0.0118658 0.022709" rpy="-0.0549698 0.711982 0.00994433"/>   calib R and T  KO- -->
-      <!-- <origin xyz="0.022 0.0225 0.0" rpy="-0.0292745 0.682572 0.0222799"/>  calib R, measured T  KO-->
-      <!-- <origin xyz="0 0.000831867 0" rpy="-0.0292745 0.682572 0.0222799"/>  calib R, zero T  KO-->
+      <origin xyz="0.0005 0.0 0.0365" rpy="0.0 0.0 0.0"/>
     </xacro:unless>
   </xtion_camera>

Commit message: Fix visual location of Xtion camera

File: thorp_description/urdf/thorp.urdf.xacro (robot description, xacro)
@@ -209,5 +209,5 @@
     <xacro:if value="$(arg simulation)">
       <origin xyz="0.022 0.003 0.002" rpy="0.0 0.694626 0.0"/>
-      <origin xyz="-0.015 0.0035 0.004" rpy="0 0 0"/>    <!-- Visual origin -->
+      <origin xyz="-0.015 -0.018 0.004" rpy="0.0 0.0 0.0"/>    <!-- Visual origin -->
     </xacro:if>
     <!-- Extrinsic parameters obtained by fitting the visible pc to robot model -->

Commit message: More precise mass for sonars array mount

File: thorp_description/urdf/thorp.urdf.xacro (robot description, xacro)
@@ -242,14 +242,8 @@
       </geometry>
     </visual>
-    <xacro:box_inertia length="0.17" width="0.325" height="0.035" mass="0.3" x="0.068"/>
-    <!-- Include also the 11 EZ2 and the arduino board: 0.22 + 11 * 0.005 + 0.025 = 0.3 -->
-    <!-- We don't need collision, as this part is mostly covered by kobuki base cylinder
-    <collision>
-      <origin xyz="0.068 0.0 0.0" rpy="0.0 0.0 0.0"/>
-      <geometry>
-        <box size="0.17 0.325 0.035"/>
-      </geometry>
-    </collision>
--->
+    <xacro:box_inertia length="0.17" width="0.325" height="0.035" mass="0.36" x="0.068"/>
+    <!-- This inertia tensor ncludes the 11 EZ2 (plus cables and mountings) and the arduino board:
+         0.22 + 11 * (0.0043 + 0.005) + 0.037 = 0.36 -->
+    <!-- We don't need collision, as this part is mostly covered by kobuki base cylinder -->
   </link>
   <xacro:macro name="LV_MaxSonar_EZ2_sensor" params="name parent x_loc y_loc yaw">

Commit message: Add a tray to the robot model

File: thorp_description/urdf/thorp.urdf.xacro (robot description, xacro)
@@ -9,4 +9,5 @@
     - 5 IR sensors
     - Turtlebot arm
+    - Tray next to it
     - Rocket launcher
     - Auxiliary 3D sensor (Creative Senz3D)
@@ -40,5 +41,5 @@
   <xacro:property name="joints_vlimit" value="0.8"/>
   <!-- <xacro:property name="pan_llimit" value="-2.617"/> -->
-  <!-- <xacro:property name="pan_ulimit" value=" 2.617"/> -->
+<!--   <xacro:property name="pan_ulimit" value=" 2.617"/>-->
   <xacro:property name="pan_llimit" value="${-M_PI/2}"/>
   <xacro:property name="pan_ulimit" value="${+M_PI/2}"/>
@@ -113,4 +114,34 @@
   </joint>
   <link name="ir_arm_link"/>
+  <!-- Tray for gathering objects -->
+  <!-- Dimensions: 150x150x15 mm; mesh base is at z=0 relative to tray_link (we can -->
+  <!-- ignore thickness, as it's only 2mm). It's supported by two bottom stack poles -->
+  <xacro:stack_bottom_pole parent="plate_top_link" number="16" x_loc=" 0.014" y_loc="-0.0516" z_loc="${0.035/2}"/>
+  <xacro:stack_bottom_pole parent="plate_top_link" number="17" x_loc=" 0.014" y_loc="-0.0980" z_loc="${0.035/2}"/>
+  <xacro:property name="tray_depth" value="0.015"/>
+  <xacro:property name="tray_side" value="0.15"/>
+  <joint name="tray_joint" type="fixed">
+    <origin xyz="0.014 -0.0748 ${0.006/2 + 0.0435}" rpy="0.0 0.0 0.0"/>
+    <parent link="plate_top_link"/>
+    <child link="tray_link"/>
+  </joint>
+  <link name="tray_link">
+    <visual>
+      <origin xyz="0.0 0.0 0.0" rpy="0.0 0.0 0.0"/>
+      <geometry>
+        <mesh filename="package://thorp_description/meshes/tray.stl" scale="${M_SCALE} ${M_SCALE} ${M_SCALE}"/>
+      </geometry>
+      <material name="Yellow">
+        <color rgba="1.0 1.0 0.0 1.0"/>
+      </material>
+    </visual>
+    <collision>
+      <origin xyz="0.0 0.0 0.0" rpy="0.0 0.0 0.0"/>
+      <geometry>
+        <mesh filename="package://thorp_description/meshes/tray.stl" scale="${M_SCALE} ${M_SCALE} ${M_SCALE}"/>
+      </geometry>
+    </collision>
+    <xacro:box_inertia length="${tray_side}" width="${tray_side}" height="${tray_depth}" mass="0.040" z="${tray_depth/2}"/>
+  </link>
   <!-- Auxiliary Senz3D camera plus mounting on Thorp -->
   <!-- Mounting poles: a pair of top poles -->
@@ -127,5 +158,5 @@
       <origin xyz="0.0075 0.0 -0.003" rpy="0.0 0.0 0.0"/>
       <geometry>
-        <mesh filename="package://thorp_description/meshes/senz3d_mount.stl" scale="0.001 0.001 0.001"/>
+        <mesh filename="package://thorp_description/meshes/senz3d_mount.stl" scale="${M_SCALE} ${M_SCALE} ${M_SCALE}"/>
       </geometry>
       <material name="Black">
@@ -190,5 +221,5 @@
       <origin xyz="0.0 0 0.0" rpy="0.0 0.0 ${M_PI/2}"/>
       <geometry>
-        <mesh filename="package://thorp_description/meshes/xtion_mount.stl" scale="0.001 0.001 0.001"/>
+        <mesh filename="package://thorp_description/meshes/xtion_mount.stl" scale="${M_SCALE} ${M_SCALE} ${M_SCALE}"/>
       </geometry>
       <material name="Black">

File: thorp_description/urdf/thorp_gazebo.urdf.xacro (robot description, xacro)
@@ -274,4 +274,5 @@
   <xacro:structural_part name="arm_mount"    color="Black"/>
   <xacro:structural_part name="opencm"       color="Black"/>
+  <xacro:structural_part name="tray"         color="Yellow"/>
   <xacro:structural_part name="cannon"       color="Black"/>
   <xacro:structural_part name="cannon_servo" color="Black"/>

Commit message: Cleanup arm joint limits and comment properly

File: thorp_description/urdf/thorp.urdf.xacro (robot description, xacro)
@@ -34,21 +34,18 @@
        camera is biased to the right; with this configuration, the arm doesn't block completely
        the camera vision of the operation space.
-       We constrain the elbow lower limit and both shoulder limits to force the arm to operate
-       always with the same gripper orientation, preventing the inefficient full turns.
-       TODO: I don't think we need to be that restrictive; do a better problem assessment.
+       Pan joint is rotated -30 degrees from the center to allow reaching the entire tray.
+       We artificially constrain the elbow lower limit to 0 to enforce planning always with the
+       same gripper orientation, preventing the inefficient full turns.
        We also use a deliberately low joints velocity limit to improve safety and precision;
        the physical limit of the AX-12 is 114 rpm (684 deg/s) -->
   <xacro:property name="joints_vlimit" value="0.8"/>
-  <!-- <xacro:property name="pan_llimit" value="-2.617"/> -->
-<!--   <xacro:property name="pan_ulimit" value=" 2.617"/>-->
-  <xacro:property name="pan_llimit" value="${-M_PI/2}"/>
-  <xacro:property name="pan_ulimit" value="${+M_PI/2}"/>
-  <xacro:property name="shoulder_llimit" value="-2.617"/>  <!-- -150 deg, but physical limit is -2.18 rad (-125 deg) -->
-  <xacro:property name="shoulder_ulimit" value=" 2.617"/>  <!-- +150 deg, but physical limit is +2.18 rad (+125 deg) -->
-  <!-- <xacro:property name="elbow_llimit" value=" -2.617"/> -->
-  <xacro:property name="elbow_llimit" value=" 0.0"/>       <!-- -150 deg, but physical limit is -2.41 rad (-138 deg) -->
-  <xacro:property name="elbow_ulimit" value=" 2.617"/>     <!-- +150 deg, but physical limit is +2.41 rad (+138 deg) -->
-  <xacro:property name="wrist_llimit" value="-1.745"/>     <!-- -100 deg -->
-  <xacro:property name="wrist_ulimit" value=" 1.745"/>     <!-- +100 deg -->
+  <xacro:property name="pan_llimit" value="${-AX12_RANGE/2 - M_PI/6}"/>  <!-- rotated -30 degrees -->
+  <xacro:property name="pan_ulimit" value="${+AX12_RANGE/2 - M_PI/6}"/>  <!-- TODO change on real robot! -->
+  <xacro:property name="shoulder_llimit" value="${-AX12_RANGE/2}"/>
+  <xacro:property name="shoulder_ulimit" value="${+AX12_RANGE/2}"/>
+  <xacro:property name="elbow_llimit" value="0.0"/>                  <!-- force constant gripper orientation -->
+  <xacro:property name="elbow_ulimit" value="${+AX12_RANGE/2}"/>
+  <xacro:property name="wrist_llimit" value="${-AX12_RANGE/3}"/>     <!-- -100 deg -->
+  <xacro:property name="wrist_ulimit" value="${+AX12_RANGE/3}"/>     <!-- +100 deg -->
   <xacro:turtlebot_arm parent="plate_top_link" color="White" gripper_color="Black"
                  pincher_gripper="false" turtlebot_gripper="true">

Commit message: Make tray higher and wider and move away from arm

File: thorp_description/urdf/thorp.urdf.xacro (robot description, xacro)
@@ -114,10 +114,10 @@
   <!-- Dimensions: 150x150x15 mm; mesh base is at z=0 relative to tray_link (we can -->
   <!-- ignore thickness, as it's only 2mm). It's supported by two bottom stack poles -->
-  <xacro:stack_bottom_pole parent="plate_top_link" number="16" x_loc=" 0.014" y_loc="-0.0516" z_loc="${0.035/2}"/>
-  <xacro:stack_bottom_pole parent="plate_top_link" number="17" x_loc=" 0.014" y_loc="-0.0980" z_loc="${0.035/2}"/>
+  <xacro:stack_bottom_pole parent="plate_top_link" number="16" x_loc=" 0.014" y_loc="-0.0576" z_loc="${0.035/2}"/>
+  <xacro:stack_bottom_pole parent="plate_top_link" number="17" x_loc=" 0.014" y_loc="-0.1250" z_loc="${0.035/2}"/>
   <xacro:property name="tray_depth" value="0.015"/>
   <xacro:property name="tray_side" value="0.15"/>
   <joint name="tray_joint" type="fixed">
-    <origin xyz="0.014 -0.0748 ${0.006/2 + 0.0435}" rpy="0.0 0.0 0.0"/>
+    <origin xyz="0.014 -0.0913 ${0.006/2 + 0.0435}" rpy="0.0 0.0 0.0"/>
     <parent link="plate_top_link"/>
     <child link="tray_link"/>

Commit message: Add holes to mount the tray and displace to match plate holes

File: thorp_description/urdf/thorp.urdf.xacro (robot description, xacro)
@@ -114,10 +114,10 @@
   <!-- Dimensions: 150x150x15 mm; mesh base is at z=0 relative to tray_link (we can -->
   <!-- ignore thickness, as it's only 2mm). It's supported by two bottom stack poles -->
-  <xacro:stack_bottom_pole parent="plate_top_link" number="16" x_loc=" 0.014" y_loc="-0.0576" z_loc="${0.035/2}"/>
-  <xacro:stack_bottom_pole parent="plate_top_link" number="17" x_loc=" 0.014" y_loc="-0.1250" z_loc="${0.035/2}"/>
+  <xacro:stack_bottom_pole parent="plate_top_link" number="16" x_loc="0.015" y_loc="-0.0585" z_loc="${0.035/2}"/>
+  <xacro:stack_bottom_pole parent="plate_top_link" number="17" x_loc="0.015" y_loc="-0.1265" z_loc="${0.035/2}"/>
   <xacro:property name="tray_depth" value="0.015"/>
   <xacro:property name="tray_side" value="0.15"/>
   <joint name="tray_joint" type="fixed">
-    <origin xyz="0.014 -0.0913 ${0.006/2 + 0.0435}" rpy="0.0 0.0 0.0"/>
+    <origin xyz="0.015 -0.0925 ${0.006/2 + 0.0435}" rpy="0.0 0.0 0.0"/>
     <parent link="plate_top_link"/>
     <child link="tray_link"/>
