Commit message: Place the tray on middle poles and remove the Senz3D

File: thorp_description/urdf/thorp.urdf.xacro (robot description, xacro)
@@ -11,5 +11,4 @@
     - Tray next to it
     - Rocket launcher
-    - Auxiliary 3D sensor (Creative Senz3D)
     - Manipulation 3D sensor (Asus Xtion Pro)
 -->
@@ -20,5 +19,4 @@
   <xacro:include filename="$(find kobuki_description)/urdf/kobuki.urdf.xacro"/>
   <xacro:include filename="$(find thorp_description)/urdf/thorp_gazebo.urdf.xacro"/>
-  <xacro:include filename="$(find thorp_description)/urdf/senz3d.urdf.xacro"/>
   <xacro:include filename="$(find thorp_description)/urdf/cannon.urdf.xacro"/>
   <xacro:include filename="$(find thorp_description)/urdf/kinect.urdf.xacro"/>
@@ -112,11 +110,11 @@
   <!-- Tray for gathering objects -->
   <!-- Dimensions: 150x150x15 mm; mesh base is at z=0 relative to tray_link (we can -->
-  <!-- ignore thickness, as it's only 2mm). It's supported by two bottom stack poles -->
-  <xacro:stack_bottom_pole parent="plate_top_link" number="16" x_loc="0.015" y_loc="-0.0585" z_loc="${0.035/2}"/>
-  <xacro:stack_bottom_pole parent="plate_top_link" number="17" x_loc="0.015" y_loc="-0.1265" z_loc="${0.035/2}"/>
+  <!-- ignore thickness, as it's only 2mm). It's supported by two middle stack poles -->
+  <xacro:stack_middle_pole parent="plate_top_link" number="16" x_loc="0.015" y_loc="-0.0585" z_loc="${0.047/2}" roll="${M_PI}"/>
+  <xacro:stack_middle_pole parent="plate_top_link" number="17" x_loc="0.015" y_loc="-0.1265" z_loc="${0.047/2}" roll="${M_PI}"/>
   <xacro:property name="tray_depth" value="0.015"/>
   <xacro:property name="tray_side" value="0.15"/>
   <joint name="tray_joint" type="fixed">
-    <origin xyz="0.015 -0.0925 ${0.006/2 + 0.0435}" rpy="0.0 0.0 0.0"/>
+    <origin xyz="0.015 -0.0925 ${0.006/2 + 0.0508}" rpy="0.0 0.0 0.0"/>
     <parent link="plate_top_link"/>
     <child link="tray_link"/>
@@ -140,9 +138,9 @@
     <xacro:box_inertia length="${tray_side}" width="${tray_side}" height="${tray_depth}" mass="0.040" z="${tray_depth/2}"/>
   </link>
-  <!-- Auxiliary Senz3D camera plus mounting on Thorp -->
-  <!-- Mounting poles: a pair of top poles -->
+  <!-- Manipulation Asus Xtion Pro camera mounted on top plate -->
+  <!-- First level of mounting poles: a pair of top poles -->
   <xacro:stack_top_pole parent="plate_top_link" number="10" x_loc="-0.1124" y_loc=" 0.098" z_loc="${0.006/2 + 0.2032/2}"/>
   <xacro:stack_top_pole parent="plate_top_link" number="20" x_loc="-0.1124" y_loc="-0.098" z_loc="${0.006/2 + 0.2032/2}"/>
-  <!-- Mounting plate -->
+  <!-- Intermediate plate to give consistence (used to be the mounting for the Senz3D camera) -->
   <joint name="senz3d_mount_joint" type="fixed">
     <origin xyz="-0.1124 0.0 ${0.006/2 + 0.2032 + 0.005/2}" rpy="0.0 0.0 0.0"/>
@@ -168,39 +166,5 @@
     <xacro:box_inertia length="0.03" width="0.22" height="0.006" mass="0.040"/>
   </link>
-  <!-- The camera itself -->
-  <joint name="senz3d_calib_joint" type="fixed">
-    <!-- Ideal extrinsic parameters obtained from robot model -->
-    <xacro:if value="$(arg simulation)">
-      <origin xyz="0.02 0.013 0.022" rpy="0.0 0.0 0.0"/>
-    </xacro:if>
-    <!-- Extrinsic parameters obtained through arm-camera calibration:
-         http://wiki.ros.org/turtlebot_arm_kinect_calibration -->
-    <!-- NOTE: Not required by now in its role of auxiliary camera -->
-    <xacro:unless value="$(arg simulation)">
-      <origin xyz="0.02 0.013 0.022" rpy="0.0 0.0 0.0"/>
-    </xacro:unless>
-    <parent link="senz3d_mount_link"/>
-    <child link="senz3d_calib_link"/>
-  </joint>
-  <link name="senz3d_calib_link"/>
-  <!-- Seems like Gazebo kinect plugin needs to use a centered frame instead of separated rgb and depth.
-       No idea if this makes any sense, but it works! I also move the optical tf a bit forward to make
-       pointcloud match better the model; this is absolutely arbitrary...
-       yay,,, I understand now better; gazebo knows nothing about optical axis, just uses camera link
-       (or whatever link u attach the plugin to) to retro-project the scene; so I need this hack to make
-       camera and optical frames match (and would need another hack without depth registration) -->
-  <xacro:if value="$(arg simulation)">
-    <joint name="senz3d_gazebo_optical_joint" type="fixed">
-      <origin xyz="0.004 0.0 0.0" rpy="${-M_PI/2} 0.0 ${-M_PI/2}"/>
-      <parent link="senz3d_link"/>
-      <child link="senz3d_gazebo_optical_frame"/>
-    </joint>
-    <link name="senz3d_gazebo_optical_frame"/>
-  </xacro:if>
-  <xacro:sensor_senz3d parent="senz3d_calib_link" name="senz3d">
-    <origin xyz="0.0 0.0 0.0" rpy="0.0 0.0 0.0"/>
-  </xacro:sensor_senz3d>
-  <!-- Manipulation Asus Xtion Pro camera mounted on top of the Senz3D's mounting plate -->
-  <!-- Mounting poles: two columns made with one top and one middle poles stacked -->
+  <!-- Second level of mounting poles: two columns made with one top and one middle poles stacked -->
   <!-- The Z loc of the lower top poles is : 1/2*plate height + 3/2*top pole height -->
   <!-- The Z loc of the upper middle poles is : 1/2*plate height + top pole height + 1/2*middle pole height (with screw) -->
@@ -209,5 +173,5 @@
   <xacro:stack_middle_pole parent="senz3d_mount_link" number="11" x_loc="0.0" y_loc=" 0.098" z_loc="${0.005/2 + 0.2032 + 0.0608/2}"/>
   <xacro:stack_middle_pole parent="senz3d_mount_link" number="21" x_loc="0.0" y_loc="-0.098" z_loc="${0.005/2 + 0.2032 + 0.0608/2}"/>
-  <!-- Mounting plate. The Z loc of the upper middle poles is: -->
+  <!-- Camera mounting plate. The Z loc of the upper middle poles is: -->
   <!--   1/2 * Senz3D mounting plate height + middle pole height (without screw) + top pole height + mounting's poles housing -->
   <joint name="xtion_mount_joint" type="fixed">
@@ -257,5 +221,12 @@
     <link name="xtion_gazebo_optical_frame"/>
   </xacro:if>        TODO: I think I can remove this because I use registered depth images
-                      yes,,, see explanation with Senz3D;  remove all this once all work on real robot too -->
+                      yes,,, see explanation with Senz3D;  remove all this once all work on real robot too
+  from Senz3D: Seems like Gazebo kinect plugin needs to use a centered frame instead of separated rgb and depth.
+       No idea if this makes any sense, but it works! I also move the optical tf a bit forward to make
+       pointcloud match better the model; this is absolutely arbitrary...
+       yay,,, I understand now better; gazebo knows nothing about optical axis, just uses camera link
+       (or whatever link u attach the plugin to) to retro-project the scene; so I need this hack to make
+       camera and optical frames match (and would need another hack without depth registration)
+                      -->
   <!-- Sonar sensors forming a half ring centered on (and slightly above) base_link -->
   <joint name="sonars_joint" type="fixed">

File: thorp_description/urdf/thorp_gazebo.urdf.xacro (robot description, xacro)
@@ -48,44 +48,4 @@
     </gazebo>
   </xacro:macro>
-  <!-- Simulated Creative Senz3d camera  DISABLE by now as Gazebo2 cannot handle 3 instances of this plugin!  TODO: retry with Gazebo5
-  <gazebo reference="senz3d_link">
-    <sensor type="depth" name="senz3d">
-      <always_on>true</always_on>
-      <update_rate>10.0</update_rate>
-      <camera>
-        <horizontal_fov>${74.0*M_PI/180.0}</horizontal_fov>
-        <image>
-          <format>B8G8R8</format>
-          <width>320</width>
-          <height>240</height>
-        </image>
-        <clip>
-          <near>0.05</near>
-          <far>1.5</far>
-        </clip>
-      </camera>
-      <plugin name="depth_camera_controller" filename="libgazebo_ros_depth_camera.so">
-        <cameraName>senz3d</cameraName>
-        <alwaysOn>true</alwaysOn>
-        <updateRate>0</updateRate>
-        <imageTopicName>rgb/image_color</imageTopicName>
-        <depthImageTopicName>depth/image_raw</depthImageTopicName>
-        <pointCloudTopicName>depth/points</pointCloudTopicName>
-        <cameraInfoTopicName>rgb/camera_info</cameraInfoTopicName>
-        <depthImageCameraInfoTopicName>depth/camera_info</depthImageCameraInfoTopicName>
-        <frameName>senz3d_gazebo_optical_frame</frameName>
-        <baseline>0.1</baseline>
-        <distortion_k1>0.0</distortion_k1>
-        <distortion_k2>0.0</distortion_k2>
-        <distortion_k3>0.0</distortion_k3>
-        <distortion_t1>0.0</distortion_t1>
-        <distortion_t2>0.0</distortion_t2>
-        <pointCloudCutoff>0.10</pointCloudCutoff>
-        <pointCloudCutoffMax>1.0</pointCloudCutoffMax>
-      </plugin>
-    </sensor>
-    <selfCollide>true</selfCollide>
-    <gravity>true</gravity>
-  </gazebo>   DISABLED -->
   <!-- LV-MaxSonar-EZ2 ultrasound sensors
        Use Hector sonar plugin to emulate the wide fov of the EZ2

Commit message: Rotate pan joint -90 instead of -30 degrees to allow reaching the entire tray. Constrain both elbow and wrist lower limit to avoid the inefficient full turns.

File: thorp_description/urdf/thorp.urdf.xacro (robot description, xacro)
@@ -31,17 +31,17 @@
        camera is biased to the right; with this configuration, the arm doesn't block completely
        the camera vision of the operation space.
-       Pan joint is rotated -30 degrees from the center to allow reaching the entire tray.
-       We artificially constrain the elbow lower limit to 0 to enforce planning always with the
-       same gripper orientation, preventing the inefficient full turns.
+       Pan joint is rotated -90 degrees from the center to allow reaching the entire tray.
+       We artificially constrain elbow and wrist lower limit to 0 to enforce planning always
+       with the same gripper orientation, preventing the inefficient full turns.
        We also use a deliberately low joints velocity limit to improve safety and precision;
        the physical limit of the AX-12 is 114 rpm (684 deg/s) -->
   <xacro:property name="joints_vlimit" value="0.8"/>
-  <xacro:property name="pan_llimit" value="${-AX12_RANGE/2 - M_PI/6}"/>  <!-- rotated -30 degrees -->
-  <xacro:property name="pan_ulimit" value="${+AX12_RANGE/2 - M_PI/6}"/>  <!-- TODO change on real robot! -->
+  <xacro:property name="pan_llimit" value="${-AX12_RANGE/2 - M_PI/2}"/>  <!-- rotated -90 degrees -->
+  <xacro:property name="pan_ulimit" value="${+AX12_RANGE/2 - M_PI/2}"/>  <!-- TODO change on real robot! -->
   <xacro:property name="shoulder_llimit" value="${-AX12_RANGE/2}"/>
   <xacro:property name="shoulder_ulimit" value="${+AX12_RANGE/2}"/>
   <xacro:property name="elbow_llimit" value="0.0"/>                  <!-- force constant gripper orientation -->
   <xacro:property name="elbow_ulimit" value="${+AX12_RANGE/2}"/>
-  <xacro:property name="wrist_llimit" value="${-AX12_RANGE/3}"/>     <!-- -100 deg -->
+  <xacro:property name="wrist_llimit" value="0.0"/>                  <!-- force constant gripper orientation -->
   <xacro:property name="wrist_ulimit" value="${+AX12_RANGE/3}"/>     <!-- +100 deg -->
   <xacro:turtlebot_arm parent="plate_top_link" color="White" gripper_color="Black"

Commit message: Fix Xtion 3D model visual

File: thorp_description/urdf/thorp.urdf.xacro (robot description, xacro)
@@ -203,11 +203,11 @@
     <xacro:if value="$(arg simulation)">
       <origin xyz="0.022 0.003 0.002" rpy="0.0 0.694626 0.0"/>
-      <origin xyz="-0.015 -0.018 0.004" rpy="0.0 0.0 0.0"/>    <!-- Visual origin -->
+      <origin xyz="-0.011 -0.022 0.0" rpy="${M_PI/2} 0.0 ${M_PI/2}"/>    <!-- make the camera 3D model match -->
     </xacro:if>
     <!-- Extrinsic parameters obtained by fitting the visible pc to robot model -->
     <xacro:unless value="$(arg simulation)">
       <origin xyz="-0.012 0.0065 -0.012" rpy="0.0 0.697357 0.0"/>
-      <!-- Visual origin corrections: undo the rotations for better aesthetics  -->
-      <origin xyz="0.0005 0.0 0.0365" rpy="0.0 0.0 0.0"/>
+      <!-- Visual origin corrections to make the camera 3D model match -->
+      <origin xyz="0.008 -0.025 0.033" rpy="${M_PI/2} 0.0 ${M_PI/2}"/>
     </xacro:unless>
   </xacro:xtion_camera>

File: thorp_description/urdf/xtion.urdf.xacro (robot description, xacro)
@@ -30,5 +30,5 @@
         <xacro:insert_block name="visual_origin"/>
         <geometry>
-          <mesh filename="package://turtlebot_description/meshes/sensors/xtion_pro_camera.dae"/>
+          <mesh filename="package://thorp_description/meshes/asus_xtion_pro_live.dae" scale="0.001 0.001 0.001"/>
         </geometry>
       </visual>
@@ -36,6 +36,6 @@
         <xacro:insert_block name="visual_origin"/>
         <geometry>
-        <box size="0.04 0.185 0.03"/>
-      </geometry>
+          <box size="0.04 0.185 0.03"/>
+        </geometry>
       </collision>
       <inertial>
