Commit message: Use xacro:insert_block as pose for the xtion collision object

File: thorp_description/urdf/xtion.urdf.xacro (robot description, xacro)
@@ -34,5 +34,5 @@
       </visual>
       <collision>
-        <origin xyz="-0.018 0.0035 0.004" rpy="0 0 0"/>
+        <xacro:insert_block name="visual_origin"/>
         <geometry>
         <box size="0.04 0.185 0.03"/>

Commit message: Scale-down the Xtion mesh

File: thorp_description/urdf/xtion.urdf.xacro (robot description, xacro)
@@ -30,5 +30,5 @@
         <xacro:insert_block name="visual_origin"/>
         <geometry>
-          <mesh filename="package://turtlebot_description/meshes/sensors/xtion_pro_camera.dae"/>
+          <mesh filename="package://turtlebot_description/meshes/sensors/xtion_pro_camera.dae" scale="${M_SCALE} ${M_SCALE} ${M_SCALE}"/>
         </geometry>
       </visual>

Commit message: Remove xtion scaling; no idea what happened but now makes the camera minuscule

File: thorp_description/urdf/xtion.urdf.xacro (robot description, xacro)
@@ -30,5 +30,5 @@
         <xacro:insert_block name="visual_origin"/>
         <geometry>
-          <mesh filename="package://turtlebot_description/meshes/sensors/xtion_pro_camera.dae" scale="${M_SCALE} ${M_SCALE} ${M_SCALE}"/>
+          <mesh filename="package://turtlebot_description/meshes/sensors/xtion_pro_camera.dae"/>
         </geometry>
       </visual>

Commit message: Make kinect launcher thorp-specific (and so much simpler)

File: thorp_description/urdf/xtion.urdf.xacro (robot description, xacro)
@@ -3,5 +3,5 @@
   <!-- Xacro properties -->
   <xacro:property name="asus_xtion_pro_depth_rel_rgb_py" value="0.0270"/>
-  <xacro:property name="asus_xtion_pro_cam_rel_rgb_py" value="-0.0220"/>
+  <xacro:property name="asus_xtion_pro_cam_rel_rgb_py" value="0.0"/>
   <!-- 3D sensor macro -->
   <xacro:macro name="xtion_camera" params="parent name *origin *visual_origin">

Commit message: Fix xtion collision model

File: thorp_description/urdf/xtion.urdf.xacro (robot description, xacro)
@@ -36,5 +36,5 @@
         <xacro:insert_block name="visual_origin"/>
         <geometry>
-          <box size="0.04 0.185 0.03"/>
+          <box size="0.185 0.03 0.04"/>  <!-- match mesh rotation of pi/2 around x and z axis -->
         </geometry>
       </collision>
